File: hardware/kicad/001_main_controller_board/Indiv_sensor.kicad_sch (KiCad schematic)
At the start: 5 parts, among them Q106 WM02N08F, U108 VCNT2025X01

Commit message: Hardware: Kicad names and schematics aligned for initial release. Added a mounting hole on the sensor board and added RS485 Bias on the main sensor board. Unnecessary files removed, readme updated.
Other:
- company: (none) -> Noah Jaffe
Changed lines of the file:
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@@
 	(paper "A4")
 	(title_block
-		(date "2025-12-04")
-		(rev "B")
+		(date "2026-04-22")
+		(rev "A")
+		(company "Noah Jaffe")
 	)
 	(text "Note: Active High"
