File: hardware/kicad/001_main_controller_board/PHOTON_main_controller.kicad_sch (KiCad schematic)
At the start: 83 parts, among them J1 FH34SRJ-18S-0.5SH(50), J102 JST_SH RS-485_1, J103 JST_SH RS-485_2, J3 USB_C_Receptacle_USB2.0, J4 Micro_SD_Card, J6 Conn_01x04, SW1 SW_Push, U1 RP2350_60QFN, U101 APS6404L-3SQR-ZR, U102 THVD1424RGTR, U2 NCP1117-3.3_SOT223, U3 W25Q128JVPIQ, U4 TPD4E05U06DQAR, Y1 ABM8-272-T3

Commit message: Consolidate symbol libraries, normalise BOM data, Rev B for all three boards
Libraries
- Move PHOTON and PHOTON_Modified to hardware/kicad/, shared by all three
  projects, replacing six divergent per-project copies. 002's versions taken
  as canonical (correct pin electrical types); 001-only parts recovered from
  the schematic cache. All 459 footprint and 464 symbol refs resolve.
- Repoint every sym-lib-table at the shared files. Nicknames unchanged, so
  002 and 001d needed no lib_id edits; only 001's stale date-named ones.
- Fix stale footprint nicknames inside the symbol libraries (footprints:,
  RP2350_60QFN_minimal:, APS6404L-3SQR-ZR:) that would have made newly
  placed parts land with unresolvable footprints.
- Reset baked-in reference designators and MPNs on six library footprints
  back to REF** and the footprint name. SOT-563_DRL0006A carried "U6",
  which would have overwritten 001d's U5 on any field-resetting update.

Footprints
- Add SON-8_3x2mm_P0.5mm: KiCad stock SON-8 with the exposed pad and its
  four paste apertures removed. The APS6404L USON-8L (JEDEC MO-229) has no
  thermal pad and 0-0.05mm standoff, so both the copper and the paste under
  the body were wrong. Replaces the easyeda2kicad footprint on U101, whose
  0.102mm mask margin also bridged all six 0.5mm-pitch mask openings.
- Mounting holes on 001 and 001d move to the photon_common keepout
  footprint, matching 002, so a screw head cannot bridge the F.Cu power
  pour to the B.Cu ground pour.
- Remove the unused TDK T3902 microphone footprint.

BOM
- Normalise values fleet-wide: Greek mu -> ascii u, strip spaces before
  units, complete truncated inductor values. Each was splitting one part
  into two BOM lines, since the fab toolkit groups on footprint+value.
- Unify JST-SH connector values so each board emits one line, not three.
  Per-connector labels moved to Description, which is not a BOM column.
- Assign part numbers to the four largest passive lines: 100nF C1525,
  1uF C52923, 1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
Parts:
- removed C103: 100nF, Capacitor_SMD:C_0402_1005Metric, symbol Device:C
- removed C104: 1μF, Capacitor_SMD:C_0402_1005Metric, symbol Device:C
- removed CR1, CR101, CR5: H7VHD3UA, Diode_SMD:D_SOD-323, symbol 2025-08-11_08-49-29:SMF5.0A
- removed D1: LED GREEN, LED_SMD:LED_0402_1005Metric, symbol Device:LED
- removed R107: 430Ω, Resistor_SMD:R_0402_1005Metric, symbol Device:R
- removed R4: 10kΩ, Resistor_SMD:R_0402_1005Metric, symbol Device:R
- removed U102: THVD1424RGTR, photon_common:QFN_24RGTR_TEX, symbol 2025-11-21_08-29-10_THVD1424RGTR:THVD1424RGTR
- removed U2: NCP1117-3.3_SOT223, Package_TO_SOT_SMD:SOT-223-3_TabPin2, symbol Regulator_Linear:NCP1117-3.3_SOT223
- removed U4: TPD4E05U06DQAR, photon_common:DQA0010A, symbol 2025-08-11_08-44-22:TPD4E05U06QDQARQ1
- added C10: 1uF, Capacitor_SMD:C_0402_1005Metric, symbol Device:C
- added C9: 100nF, Capacitor_SMD:C_0402_1005Metric, symbol Device:C
- added CR1: PTVSHC3D7VU, photon_common:SOD-323_L1.8-W1.3-LS2.5-RD, symbol PHOTON:PTVSHC3D7VU
- added D12: D_TVS, Diode_SMD:D_SOD-523, symbol Device:D_Schottky
- added L2: 1uH, Inductor_SMD:L_1008_2520Metric, symbol Device:L
- added R103: 100kΩ, Resistor_SMD:R_0402_1005Metric, symbol Device:R
- added R104, R105: 200kΩ, Resistor_SMD:R_0402_1005Metric, symbol Device:R
- added U4: TPD4E05U06DQAR, photon_common:DQA0010A, symbol PHOTON:TPD4E05U06QDQARQ1
- added U5: THVD1424RGTR, photon_common:QFN_24RGTR_TEX, symbol PHOTON:THVD1424RGTR
- added U6: TPS62A0569ADRLR, photon_common:SOT-563_DRL0006A, symbol PHOTON:TPS62A0569ADRLR
- C1: value 10uF -> 4.7uF; JLCPCB Part # (none) -> C1779
- C101, C105, C107, C13, C14, C15, C16, C19, C20, C21, C22, C5, C8: JLCPCB Part # (none) -> C1525
- C102, C106, C108: value 1μF -> 1uF; JLCPCB Part # (none) -> C52923
- C17, C18: JLCPCB Part # (none) -> C1548
- C4: value 10uF -> 22uF; JLCPCB Part # (none) -> C45783
- C58: JLCPCB Part # (none) -> C1523
- D2: footprint LED_SMD:LED_0402_1005Metric -> LED_SMD:LED_0603_1608Metric; JLCPCB Part # C130719 -> C2286
- D3: value LED GREEN -> LED RED; footprint LED_SMD:LED_0402_1005Metric -> LED_SMD:LED_0603_1608Metric; JLCPCB Part # C130722 -> C2286
- FB1: JLCPCB Part # C1002 -> C14709
- H101, H102, H103, H104: footprint MountingHole:MountingHole_2.7mm_M2.5_ISO7380 -> photon_common:MountingHole_2.7mm_M2.5_Keepout
- J102: value JST_SH RS-485_1 -> JST_SH
- J103: value JST_SH RS-485_2 -> JST_SH
- J3: symbol Connector:USB_C_Receptacle_USB2.0 -> PHOTON_Modified:USB_C_Receptacle_USB2.0
- J4: symbol Connector:Micro_SD_Card -> PHOTON_Modified:Micro_SD_Card
- J6: value Conn_01x04 -> JST_SH
- L1: value 3.3u -> 3.3uH
- R1: value 1MΩ -> 0Ω; footprint Resistor_SMD:R_0805_2012Metric_Pad1.20x1.40mm_HandSolder -> Resistor_SMD:R_0402_1005Metric
- R10: value 10 kΩ -> 10kΩ
- R106: value 430Ω -> 51kΩ
- R2, R3: value 5.1 kΩ -> 5.1kΩ
- R5: value 22kΩ -> 10kΩ
- U1: symbol MCU_RaspberryPi_RP2350:RP2350_60QFN -> PHOTON:RP2350_60QFN
- U101: footprint photon_common:PSON50P200X300X50-9N -> photon_common:SON-8_3x2mm_P0.5mm; symbol APS6404L-3SQR-ZR:APS6404L-3SQR-ZR -> PHOTON:APS6404L-3SQR-ZR; Availability (none) -> Not in stock; Description_1 (none) -> DRAM IoT RAM 64Mb QSPI (x1,x4) SDR 133/84MHz, RBX, 3V, USON8; MP (none) -> APS6404L-3SQR-ZR
- U3: symbol Memory_Flash:W25Q128JVS -> PHOTON:W25Q128JVS
- Y1: symbol Device:Crystal_GND24 -> PHOTON_Modified:Crystal_GND24
- renumbered R104 to R13, R105 to R4, R103 to R9
Connections:
- net +3V3: now also C10.1, C9.1, D12.1 (K), L2.2, R104.2, U5.13 (VIO), U5.14 (VCC), U5.15 (H/F); no longer J102.2 (Pin_2), J103.2 (Pin_2), R106.2
- net GND: now also C10.2, C9.2, CR1.2 (A), D12.2 (A), R103.2, U4.3 (GND), U4.8 (GND), U5.17 (GND), U5.6 (GND), U6.2 (GND)
- net GPIO1: now also U5.2 (RE), U5.3 (DE)
- net GPIO18: now also U5.5 (TERM_TX), U5.7 (TERM_RX)
- net RS485_N: now also U5.10 (Z)
- net RS485_P: now also U5.9 (Y); no longer R106.1
- net UART_RX: now also U5.1 (R)
- net UART_TX: now also U5.4 (D)
- net USB_D+: now also U4.4 (D2+), U4.7 (NC)
- net USB_D-: now also U4.5 (D2-), U4.6 (NC)
- net at J3.A5 (CC1), R2.2: now also U4.1 (D1+), U4.10 (NC)
- net at C1.1, FB1.2: now also U6.3 (VIN), U6.5 (EN)
- net at J3.B5 (CC2), R3.2: now also U4.2 (D1-), U4.9 (NC)
- net at R1.2: now also J3.SH (SHIELD); no longer J3.S1 (SHIELD)
- net VBUS renamed +5V
- net +5V: now also J102.2 (Pin_2), J103.2 (Pin_2), CR1.1 (K)
- new net: R103.1, R106.1, U6.1 (FB)
- new net: R105.1, R106.2
- new net: R104.1, R105.2
- new net: L2.1, U6.4 (SW)
- no-connect marks 13 -> 15
Other:
- note added: "3.3V I2C"
- note added: "For proof of concepts"
- note removed: "For debug and simple proof of concepts"
- note removed: "RS485 Differential Bias. One per bus."
- note removed: "RS485 needs a termination at the end of the bus. A middle device with both left and right connected needs to have both ends unterminated. But if it's at the end of the bus, and JST right is used, then drive RS485_TERM high. If end-fed by JST left, then right must be terminated"
- moved on the sheet: C101, C102, C21, J102, J103, J6, R13, R4, R7, R8, R9, SW1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

Commit message: Pin the 4.7uF 0402 to C23733 across all three boards
JLCPCB selected Samsung CL05A475MP5NRNC (4.7uF 10V X5R +/-20% 0402) for the
blank 4.7uF line when 001d and 002 were ordered. Recording it so the choice is
deterministic on the next order rather than made again at upload time, possibly
differently.

Matched on value AND footprint: the twelve 0402 parts (C2/C3/C6/C7 on each
board, across both the standard and small-pads variants) take C23733, while
C1 — the 4.7uF 0805 at the buck input — keeps C1779.

10 V is the right side of the choice for a 3.3 V rail; a 6.3 V part would
derate much harder under bias. These four are bypass and the low-bias +1V1
core rail, not the buck's control loop, which hangs off C4 (22uF 0805).

Co-Authored-By: Claude Opus 5 <noreply@anthropic.com>
Parts:
- C2, C3, C6, C7: JLCPCB Part # (none) -> C23733
Changed lines of the file:
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@@
 			)
 		)
+		(property "JLCPCB Part #" "C23733"
+			(at 0 0 0)
+			(show_name no)
+			(do_not_autoplace no)
+			(hide yes)
+			(effects
+				(font
+					(size 1.27 1.27)
+				)
+			)
+		)
 		(property "Description" ""
 			(at 237.49 29.21 0)
@@
 			)
 		)
+		(property "JLCPCB Part #" "C23733"
+			(at 0 0 0)
+			(show_name no)
+			(do_not_autoplace no)
+			(hide yes)
+			(effects
+				(font
+					(size 1.27 1.27)
+				)
+			)
+		)
 		(property "Description" ""
 			(at 190.5 67.31 0)
@@
 			)
 		)
+		(property "JLCPCB Part #" "C23733"
+			(at 0 0 0)
+			(show_name no)
+			(do_not_autoplace no)
+			(hide yes)
+			(effects
+				(font
+					(size 1.27 1.27)
+				)
+			)
+		)
 		(property "Description" ""
 			(at 236.22 54.61 0)
@@
 			(effects
 				(font
+					(size 1.27 1.27)
+				)
+			)
+		)
+		(property "JLCPCB Part #" "C23733"
+			(at 0 0 0)
+			(show_name no)
+			(do_not_autoplace no)
+			(hide yes)
+			(effects
+				(font
