File: hardware/kicad/002_sensor_board_example/002_Sensor_PI_RS485 board.kicad_sch (KiCad schematic)
At the start: 61 parts, among them J1 JST_SH, J2 JST_SH, J3 USB_C_Receptacle_USB2.0, SW1 SW_SPST, SW2 SW_SPST, U1 RP2350_60QFN, U2 NCP1117-3.3_SOT223, U3 W25Q128JVPIQ, U4 TPD4E05U06DQAR, U5 THVD1424RGTR, Y1 ABM8-272-T3

Commit message: 001d bumped to 5V RS485 bus voltage. Sensor board schematic cleaned up, layout not begun
Parts:
- removed C22: 100nF, Capacitor_SMD:C_0402_1005Metric, symbol Device:C
- removed JP2: SolderJumper_2_Bridged, Jumper:SolderJumper-2_P1.3mm_Bridged_RoundedPad1.0x1.5mm, symbol Jumper:SolderJumper_2_Bridged
- removed R15: DNF, Resistor_SMD:R_0402_1005Metric, symbol Device:R
- removed R17: 100kΩ, Resistor_SMD:R_0402_1005Metric, symbol Device:R
- removed R4: 120 Ω, Resistor_SMD:R_0402_1005Metric, symbol Device:R
- removed SW1, SW2: SW_SPST, footprints:SW-TH_MSK12C02, symbol spst:MSK12C02
- removed U2: NCP1117-3.3_SOT223, Package_TO_SOT_SMD:SOT-223-3_TabPin2, symbol Regulator_Linear:NCP1117-3.3_SOT223
- removed U3: W25Q128JVPIQ, footprints:WSON_128JVPIQ_WIN, symbol Memory_Flash:W25Q128JVS
- added D1: SS14, Diode_SMD:D_SMA, symbol Device:D_Schottky
- added H10, H11, H12, H13, H14, H15, H16, H5, H6, H7, H8, H9: MountingHole, MountingHole:MountingHole_2.7mm_M2.5, symbol Mechanical:MountingHole
- added JP1, JP2: SolderJumper_2_Open, symbol Jumper:SolderJumper_2_Open
- added L2: 1 uH, Inductor_SMD:L_1008_2520Metric, symbol Device:L
- added R103: 100kΩ, Resistor_SMD:R_0402_1005Metric, symbol Device:R
- added R104: 300kΩ, Resistor_SMD:R_0402_1005Metric, symbol Device:R
- added R105: 150kΩ, Resistor_SMD:R_0402_1005Metric, symbol Device:R
- added R5: 120 Ω, Resistor_SMD:R_0402_1005Metric, symbol Device:R
- added U6: TPS62A0569ADRLR, Pretty Custom:DRL0006A-MFG, symbol TI BUCK:TPS62A0569ADRLR
- C1: value 10uF -> 4.7uF; JLCPCB Part # (none) -> C1779; Part # (none) -> CL21A475KAQNNNE
- C4: value 10uF -> 22uF; JLCPCB Part # (none) -> C45783
- U1: value RP2350_60QFN -> RP2354_60QFN; JLCPCB Part # C42411118 -> C41378174
- renumbered JP101 to JP4, R101 to R4
Connections:
- net +3V3: now also L2.2, R104.1; no longer CR2.1 (K), J1.2 (Pin_2), J2.2 (Pin_2)
- net GND: now also R103.2, U6.2 (GND)
- net RS485_N: now also R4.2, R5.2
- net RS485_P: now also JP1.1 (A), JP2.1 (A); no longer R4.2
- net VBUS: now also CR2.1 (K), J1.2 (Pin_2), J2.2 (Pin_2), D1.1 (K), D1.2 (A)
- net at C1.1, FB1.2: now also U6.3 (VIN), U6.5 (EN)
- net at R4.1: now also JP1.2 (B)
- net FLASH_SS renamed QSPI_SS
- new net: R104.2, R105.1
- new net: R103.1, R105.2, U6.1 (FB)
- new net: L2.1, U6.4 (SW)
- new net: JP2.2 (B), R5.1
- no-connect marks 7 -> 6
Other:
- note added: "This built-in RS485 termination should not be used. Rather, terminate at the end of the board using the jumpers."
- note removed: "Cut for backpower issues when USB power is not used. Note: When cut, board is no longer able to be powered by USB."
- note removed: "Flash"
- note removed: "Terminate (right position) when connector is not used."
- note removed: "This built-in RS485 termination should not be used. Rather, terminate at the end of the board using the switches."
- title: PHOTON Sensor Board - 002 -> PHOTON Sensor Board - A007
- moved on the sheet: C17, C18, CR1, D3, J1, J2, J4, R18, R4, R7, R8, U4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
