File: hardware/kicad/002_sensor_board_example/4_Sensor_Bank.kicad_sch (KiCad schematic)
At the start: 9 parts, among them U401 TLA2518IRTER

Commit message: Main Controller Board (1D) now added. Cheaper design, with RP2354, and BUCK PMIC
Parts:
- removed C401, C402, C403: 1 uF, Capacitor_SMD:C_0402_1005Metric, symbol Device:C
- removed C404, C405, C406, C407: 1 nF, Capacitor_SMD:C_0402_1005Metric, symbol Device:C
- removed R401: 47k, Resistor_SMD:R_0402_1005Metric, symbol Device:R
- removed U401: TLA2518IRTER, footprints:WQFN16_RTE_TEX, symbol tla2518:TLA2518IRTER
Other:
- removed sheet Individual Sensor
- removed sheet Individual Sensor1
- removed sheet Individual Sensor2
- removed sheet Individual Sensor3
- note removed: "Place these caps next to ADC input pins"
- company: (none) -> Noah Jaffe
- title: 4 to 1 Channel Sensor Array -> (none)

Commit message: 001d bumped to 5V RS485 bus voltage. Sensor board schematic cleaned up, layout not begun
Parts:
- added C401, C402, C403: 1 uF, Capacitor_SMD:C_0402_1005Metric, symbol Device:C
- added C404, C405, C406, C407: 1 nF, Capacitor_SMD:C_0402_1005Metric, symbol Device:C
- added R401: 47k, Resistor_SMD:R_0402_1005Metric, symbol Device:R
- added U401: TLA2518IRTER, footprints:WQFN16_RTE_TEX, symbol tla2518:TLA2518IRTER
Connections:
- new net: C402.1, U401.8 (DECAP)
- new net +3V3: C401.1, C403.1, R401.1, U401.10 (DVDD), U401.7 (AVDD)
- new net BANK_CS: R401.2, U401.11 (*CS)
- new net EN0: U401.5 (AIN6/GPIO6)
- new net EN1: U401.3 (AIN4/GPIO4)
- new net EN2: U401.1 (AIN2/GPIO2)
- new net EN3: U401.15 (AIN0/GPIO0)
- new net GND: C401.2, C402.2, C403.2, C404.2, C405.2, C406.2, C407.2, U401.17 (GND), U401.9 (GND)
- new net SPI_MISO: U401.12 (SDO)
- new net SPI_MOSI: U401.14 (SDI)
- new net SPI_SCLK: U401.13 (SCLK)
- new net Y0: C404.1, U401.6 (AIN7/GPIO7)
- new net Y1: C405.1, U401.4 (AIN5/GPIO5)
- new net Y2: C406.1, U401.2 (AIN3/GPIO3)
- new net Y3: C407.1, U401.16 (AIN1/GPIO1)
Other:
- added sheet Individual Sensor (Indiv_sensor.kicad_sch)
- added sheet Individual Sensor1 (Indiv_sensor.kicad_sch)
- added sheet Individual Sensor2 (Indiv_sensor.kicad_sch)
- added sheet Individual Sensor3 (Indiv_sensor.kicad_sch)
- note added: "Place these caps next to ADC input pins"
- company: Noah Jaffe -> (none)
- title: (none) -> 4 to 1 Channel Sensor Array
