File: hardware/kicad/002_sensor_board_example/4_Sensor_Bank.kicad_sch (KiCad schematic)
At the start: 9 parts, among them U401 TLA2518IRTER

Commit message: 002 sensor board: 5V bus rework, library consolidation, DRC pass
Board (002):
- Remove SS14 bridging diode; USB-C VBUS and JST V+ are now one net.
  Worst case is back-powering a host's VBUS, acceptable in a uniform
  5V fleet, and it drops 185mW in the bridging case.
- Remove the 8x 47k CS pull-ups. At 47k they parked the TLA2518 CS
  inputs mid-rail (1.7-2.1V, between VIL 0.99 and VIH 2.31); the
  internal pull-down now defines them cleanly low. Firmware must drive
  CS high before configuring SPI.
- 5V pour along the bottom edge, 3.3V moved up to the mounting rail.
- USB-C relocated; ~200mm D+/D- run on F.Cu over the B.Cu GND pour.
- Screw-head keepouts on all mounting holes.
- Board grown 2mm in Y -> 413.66 x 35.00 mm.

Net classes:
- USB_DIFF_90 -> USB_FS, diff pair 0.8/0.15 -> 0.35/0.15. The old name
  claimed 90 ohm; on a 1.51mm 2-layer stackup it is ~140 ohm and cannot
  be otherwise. Irrelevant at Full Speed.
- Add PWR_5V (+5V) and RS485 (/RS485_P, /RS485_N).
- Restore the +3V3 -> VCC assignment lost during the rename.

Libraries:
- footprints/ -> footprints.pretty/ so KiCad will save into it.
- Consolidate symbols into PHOTON / PHOTON_Modified on 001d and 002;
  drop unused vendor-exported libraries.
- Add mousebite_34mm: 17x 1.2mm NPTH at 2mm pitch. 0.8mm webs cut more
  easily than the old 1.4mm and still pass a 0.3mm trace.
- Fix MountingHole_2.7mm_M2.5_Keepout: it disallowed pads, so each hole
  flagged its own NPTH (17 DRC errors).

Fab outputs now tracked via .gitignore negation for production/*.csv.

Co-Authored-By: Claude Opus 5 <noreply@anthropic.com>
Parts:
- removed R401: 47k, Resistor_SMD:R_0402_1005Metric, symbol Device:R
- U401: symbol tla2518:TLA2518IRTER -> PHOTON:TLA2518IRTER
Other:
- company: (none) -> Noah Jaffe
Changed lines of the file:
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@@
 	(title_block
 		(title "4 to 1 Channel Sensor Array")
-		(date "2026-01-02")
-		(rev "C")
+		(date "2026-04-22")
+		(rev "B")
+		(company "Noah Jaffe")
 	)
 	(text "Place these caps next to ADC input pins"
@@
 		(color 0 0 0 0)
 	)
-	(junction
-		(at 181.61 135.89)
-		(diameter 0)
-		(color 0 0 0 0)
-	)
 	(wire
 		(pts
@@
 	(wire
 		(pts
-			(xy 181.61 135.89) (xy 160.02 135.89)
+			(xy 160.02 135.89) (xy 184.15 135.89)
 		)
 		(stroke
@@
 		(pts
 			(xy 160.02 138.43) (xy 163.83 138.43)
-		)
-		(stroke
-			(width 0)
-			(type default)
-		)
-	)
-	(wire
-		(pts
-			(xy 184.15 135.89) (xy 181.61 135.89)
 		)
 		(stroke
@@
 	)
 	(symbol
-		(lib_id "power:VCC")
-		(at 181.61 128.27 0)
-		(unit 1)
-		(body_style 1)
-		(exclude_from_sim no)
-		(in_bom yes)
-		(on_board yes)
-		(in_pos_files yes)
-		(dnp no)
-		(property "Reference" "#PWR0404"
-			(at 181.61 132.08 0)
-			(hide yes)
-			(show_name no)
-			(do_not_autoplace no)
-			(effects
-				(font
-					(size 1.27 1.27)
-				)
-			)
-		)
-		(property "Value" "+3V3"
-			(at 180.086 124.206 0)
-			(show_name no)
-			(do_not_autoplace no)
-			(effects
-				(font
-					(size 1.27 1.27)
-				)
-			)
-		)
-		(property "Footprint" ""
-			(at 181.61 128.27 0)
-			(hide yes)
-			(show_name no)
-			(do_not_autoplace no)
-			(effects
-				(font
-					(size 1.27 1.27)
-				)
-			)
-		)
-		(property "Datasheet" ""
-			(at 181.61 128.27 0)
-			(hide yes)
-			(show_name no)
-			(do_not_autoplace no)
-			(effects
-				(font
-					(size 1.27 1.27)
-				)
-			)
-		)
-		(property "Description" "Power symbol creates a global label with name \"VCC\""
-			(at 181.61 128.27 0)
-			(hide yes)
-			(show_name no)
-			(do_not_autoplace no)
-			(effects
-				(font
-					(size 1.27 1.27)
-				)
-			)
-		)
-		(pin "1"
-		)
-		(instances
-			(project "002_Sensor_PI_RS485 board"
-				(path "/b0089fb8-2318-4750-8145-7647caa10afa/8abbdb56-ea85-4864-aa21-196a08be6eef/1f3c5546-2135-48f1-a4dc-e0c99dc1341d"
-					(reference "#PWR0404")
-					(unit 1)
-				)
-				(path "/b0089fb8-2318-4750-8145-7647caa10afa/8abbdb56-ea85-4864-aa21-196a08be6eef/25c23f8c-98d8-4cf3-af53-bf3a2aa69c0d"
-					(reference "#PWR03308")
-					(unit 1)
-				)
-				(path "/b0089fb8-2318-4750-8145-7647caa10afa/8abbdb56-ea85-4864-aa21-196a08be6eef/70b52523-2629-4084-a9e1-582b7135575b"
-					(reference "#PWR01308")
-					(unit 1)
-				)
-				(path "/b0089fb8-2318-4750-8145-7647caa10afa/8abbdb56-ea85-4864-aa21-196a08be6eef/8d30b6fc-4531-43a8-bd91-9e6b22228f4d"
-					(reference "#PWR02808")
-					(unit 1)
-				)
-				(path "/b0089fb8-2318-4750-8145-7647caa10afa/8abbdb56-ea85-4864-aa21-196a08be6eef/a2963094-a324-44eb-aae5-350c5ae995ee"
-					(reference "#PWR02308")
-					(unit 1)
-				)
-				(path "/b0089fb8-2318-4750-8145-7647caa10afa/8abbdb56-ea85-4864-aa21-196a08be6eef/a8414ea3-1864-4085-b09d-ba1ee86ddb1a"
-					(reference "#PWR0808")
-					(unit 1)
-				)
-				(path "/b0089fb8-2318-4750-8145-7647caa10afa/8abbdb56-ea85-4864-aa21-196a08be6eef/ac3e6ed6-395a-4fc3-a422-0b68eeab2252"
-					(reference "#PWR01808")
-					(unit 1)
-				)
-			)
-		)
-	)
-	(symbol
-		(lib_id "Device:R")
-		(at 181.61 132.08 0)
-		(unit 1)
-		(body_style 1)
-		(exclude_from_sim no)
-		(in_bom yes)
-		(on_board yes)
-		(in_pos_files yes)
-		(dnp no)
-		(fields_autoplaced yes)
-		(property "Reference" "R401"
-			(at 184.15 130.8099 0)
-			(show_name no)
-			(do_not_autoplace no)
-			(effects
-				(font
-					(size 1.27 1.27)
-				)
-				(justify left)
-			)
-		)
-		(property "Value" "47k"
-			(at 184.15 133.3499 0)
-			(show_name no)
-			(do_not_autoplace no)
-			(effects
-				(font
-					(size 1.27 1.27)
-				)
-				(justify left)
-			)
-		)
-		(property "Footprint" "Resistor_SMD:R_0402_1005Metric"
-			(at 179.832 132.08 90)
-			(hide yes)
-			(show_name no)
-			(do_not_autoplace no)
-			(effects
-				(font
-					(size 1.27 1.27)
-				)
-			)
-		)
-		(property "Datasheet" ""
-			(at 181.61 132.08 0)
-			(hide yes)
-			(show_name no)
-			(do_not_autoplace no)
-			(effects
-				(font
-					(size 1.27 1.27)
-				)
-			)
-		)
-		(property "Description" "Resistor"
-			(at 181.61 132.08 0)
-			(hide yes)
-			(show_name no)
-			(do_not_autoplace no)
-			(effects
-				(font
-					(size 1.27 1.27)
-				)
-			)
-		)
-		(pin "1"
-		)
-		(pin "2"
-		)
-		(instances
-			(project "002_Sensor_PI_RS485 board"
-				(path "/b0089fb8-2318-4750-8145-7647caa10afa/8abbdb56-ea85-4864-aa21-196a08be6eef/1f3c5546-2135-48f1-a4dc-e0c99dc1341d"
-					(reference "R401")
-					(unit 1)
-				)
-				(path "/b0089fb8-2318-4750-8145-7647caa10afa/8abbdb56-ea85-4864-aa21-196a08be6eef/25c23f8c-98d8-4cf3-af53-bf3a2aa69c0d"
-					(reference "R3301")
-					(unit 1)
-				)
-				(path "/b0089fb8-2318-4750-8145-7647caa10afa/8abbdb56-ea85-4864-aa21-196a08be6eef/70b52523-2629-4084-a9e1-582b7135575b"
-					(reference "R1301")
-					(unit 1)
-				)
-				(path "/b0089fb8-2318-4750-8145-7647caa10afa/8abbdb56-ea85-4864-aa21-196a08be6eef/8d30b6fc-4531-43a8-bd91-9e6b22228f4d"
-					(reference "R2801")
-					(unit 1)
-				)
-				(path "/b0089fb8-2318-4750-8145-7647caa10afa/8abbdb56-ea85-4864-aa21-196a08be6eef/a2963094-a324-44eb-aae5-350c5ae995ee"
-					(reference "R2301")
-					(unit 1)
-				)
-				(path "/b0089fb8-2318-4750-8145-7647caa10afa/8abbdb56-ea85-4864-aa21-196a08be6eef/a8414ea3-1864-4085-b09d-ba1ee86ddb1a"
-					(reference "R801")
-					(unit 1)
-				)
-				(path "/b0089fb8-2318-4750-8145-7647caa10afa/8abbdb56-ea85-4864-aa21-196a08be6eef/ac3e6ed6-395a-4fc3-a422-0b68eeab2252"
-					(reference "R1801")
-					(unit 1)
-				)
-			)
-		)
-	)
-	(symbol
 		(lib_id "power:GND")
 		(at 168.91 153.67 0)
@@
 	)
 	(symbol
-		(lib_id "tla2518:TLA2518IRTER")
+		(lib_id "PHOTON:TLA2518IRTER")
 		(at 93.98 120.65 0)
 		(unit 1)

Commit message: 002: ERC/DRC to zero, symbol and value cleanup
Schematic (ERC 24 -> 0):
- VCNT2020 renamed to VCNT2025X01, matching the part actually fitted.
  Pin types preserved: passive / open_collector / passive / passive.
  The old auto-generated VCNT2025X01 symbol (all pins Unspecified) is gone.
- THVD1424RGTR: 10 pins off Unspecified (R, RE, DE, D, TERM_TX, TERM_RX,
  Y, Z, VIO, H/F). VIO was typed as a signal despite being a supply pin.
- TLA2518IRTER: DECAP -> Passive, clearing 8 warnings at once.
- PWR_FLAG moved off J3's VBUS (which J3 already drives as a Power output)
  onto GND, which had none. One move, two errors.
- JP1/JP2/JP4 repointed to stock Jumper:SolderJumper_2_Open. The project
  copy was KiCad's older stock symbol, not a deliberate modification.
- R1 1M -> 0 ohm, bonding the USB-C shell to GND. A lone 1M is a static
  bleed, not a shield connection: open at every frequency that matters,
  and it isolated nothing since J3's GND pins are already bonded.

Layout:
- MountingHole keepout had (pads not_allowed), so each hole flagged its
  own NPTH. Fixed and patched into all 17 instances.
- Mousebite silkscreen removed (library + all 3 placements). The dashed
  line crossed the pours end to end and caused ~61 of the DRC warnings.
- 30 duplicate vias deleted. Each pair was 1 nm apart from a float->int
  round-trip in the layout plugin, so KiCad's "delete redundant vias"
  could not see them while DRC's co-located check could.
- min_resolved_spokes 2 -> 1; single-spoke pads are accepted on this
  board rather than excluded per-violation.

BOM hygiene:
- Component values normalised: no space before units, ASCII u instead of
  U+03BC, and 3.3u given its missing unit. Merges 100 kohm/100kohm and
  1 uF/1uF, which would otherwise export as separate lines for identical
  parts. 181 edits across schematics and PCB, kept in sync.

Libraries:
- PHOTON_Modified reduced to the two symbols that genuinely diverge from
  stock: Crystal_GND24 and USB_C_Receptacle_USB2.0.

Known o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
Parts:
- C401, C402, C403: value 1 uF -> 1uF
- C404, C405, C406, C407: value 1 nF -> 1nF
Changed lines of the file:
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@@
 			)
 		)
-		(property "Value" "1 uF"
+		(property "Value" "1uF"
 			(at 163.322 152.146 0)
 			(show_name no)
@@
 			)
 		)
-		(property "Value" "1 uF"
+		(property "Value" "1uF"
 			(at 93.726 144.526 0)
 			(show_name no)
@@
 			)
 		)
-		(property "Value" "1 nF"
+		(property "Value" "1nF"
 			(at 204.978 131.318 0)
 			(show_name no)
@@
 			)
 		)
-		(property "Value" "1 nF"
+		(property "Value" "1nF"
 			(at 232.918 131.318 0)
 			(show_name no)
@@
 			)
 		)
-		(property "Value" "1 nF"
+		(property "Value" "1nF"
 			(at 218.948 131.318 0)
 			(show_name no)
@@
 			)
 		)
-		(property "Value" "1 nF"
+		(property "Value" "1nF"
 			(at 245.618 131.318 0)
 			(show_name no)
@@
 			)
 		)
-		(property "Value" "1 uF"
+		(property "Value" "1uF"
 			(at 82.55 145.034 0)
 			(show_name no)
