File: hardware/kicad/002_sensor_board_example/Sensor_Array.kicad_sch (KiCad schematic)
At the start: 0 parts

Commit message: Main Controller Board (1D) now added. Cheaper design, with RP2354, and BUCK PMIC
Other:
- company: (none) -> Noah Jaffe
Changed lines of the file:
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@@
 (kicad_sch
-	(version 20250114)
+	(version 20260306)
 	(generator "eeschema")
-	(generator_version "9.0")
+	(generator_version "10.0")
 	(paper "A4")
 	(title_block
 		(title "8x4-Channel LED Sensor Array")
-		(date "2026-01-02")
-		(rev "C")
+		(date "2026-04-22")
+		(rev "E")
+		(company "Noah Jaffe")
 		(comment 1 "SPI Sensor Bank Connections")
 	)
@@
 		)
 		(fill
-			(color 0 0 0 0.0000)
+			(color 0 0 0 0)
 		)
 		(property "Sheetname" "4_Sensor_bank"
 			(at 21.59 36.1184 0)
+			(show_name no)
+			(do_not_autoplace no)
 			(effects
 				(font
@@
 		(property "Sheetfile" "4_Sensor_Bank.kicad_sch"
 			(at 21.59 57.7346 0)
+			(show_name no)
+			(do_not_autoplace no)
 			(effects
 				(font
@@
 		(property "Field2" ""
 			(at 21.59 36.83 0)
+			(show_name no)
+			(do_not_autoplace no)
 			(effects
 				(font
@@
 		)
 		(instances
-			(project "014_Sensor_PI_RS485 board"
+			(project "002_Sensor_PI_RS485 board"
 				(path "/b0089fb8-2318-4750-8145-7647caa10afa/8abbdb56-ea85-4864-aa21-196a08be6eef"
 					(page "4")
@@
 		)
 		(fill
-			(color 0 0 0 0.0000)
+			(color 0 0 0 0)
 		)
 		(property "Sheetname" "4_Sensor_bank6"
 			(at 74.93 91.9984 0)
+			(show_name no)
+			(do_not_autoplace no)
 			(effects
 				(font
@@
 		(property "Sheetfile" "4_Sensor_Bank.kicad_sch"
 			(at 74.93 113.6146 0)
+			(show_name no)
+			(do_not_autoplace no)
 			(effects
 				(font
@@
 		(property "Field2" ""
 			(at 74.93 92.71 0)
+			(show_name no)
+			(do_not_autoplace no)
 			(effects
 				(font
@@
 		)
 		(instances
-			(project "014_Sensor_PI_RS485 board"
+			(project "002_Sensor_PI_RS485 board"
 				(path "/b0089fb8-2318-4750-8145-7647caa10afa/8abbdb56-ea85-4864-aa21-196a08be6eef"
 					(page "33")
@@
 		)
 		(fill
-			(color 0 0 0 0.0000)
+			(color 0 0 0 0)
 		)
 		(property "Sheetname" "4_Sensor_bank2"
 			(at 21.59 91.9984 0)
+			(show_name no)
+			(do_not_autoplace no)
 			(effects
 				(font
@@
 		(property "Sheetfile" "4_Sensor_Bank.kicad_sch"
 			(at 21.59 113.6146 0)
+			(show_name no)
+			(do_not_autoplace no)
 			(effects
 				(font
@@
 		(property "Field2" ""
 			(at 21.59 92.71 0)
+			(show_name no)
+			(do_not_autoplace no)
 			(effects
 				(font
@@
 		)
 		(instances
-			(project "014_Sensor_PI_RS485 board"
+			(project "002_Sensor_PI_RS485 board"
 				(path "/b0089fb8-2318-4750-8145-7647caa10afa/8abbdb56-ea85-4864-aa21-196a08be6eef"
 					(page "13")
@@
 		)
 		(fill
-			(color 0 0 0 0.0000)
+			(color 0 0 0 0)
 		)
 		(property "Sheetname" "Last_sensor_bank"
 			(at 74.93 121.2084 0)
+			(show_name no)
+			(do_not_autoplace no)
 			(effects
 				(font
@@
 		(property "Sheetfile" "last_sensor_bank.kicad_sch"
 			(at 74.93 144.0946 0)
+			(show_name no)
+			(do_not_autoplace no)
 			(effects
 				(font
@@
 		)
 		(instances
-			(project "014_Sensor_PI_RS485 board"
+			(project "002_Sensor_PI_RS485 board"
 				(path "/b0089fb8-2318-4750-8145-7647caa10afa/8abbdb56-ea85-4864-aa21-196a08be6eef"
 					(page "38")
@@
 		)
 		(fill
-			(color 0 0 0 0.0000)
+			(color 0 0 0 0)
 		)
 		(property "Sheetname" "4_Sensor_bank5"
 			(at 74.93 64.0584 0)
+			(show_name no)
+			(do_not_autoplace no)
 			(effects
 				(font
@@
 		(property "Sheetfile" "4_Sensor_Bank.kicad_sch"
 			(at 74.93 85.6746 0)
+			(show_name no)
+			(do_not_autoplace no)
 			(effects
 				(font
@@
 		(property "Field2" ""
 			(at 74.93 64.77 0)
+			(show_name no)
+			(do_not_autoplace no)
 			(effects
 				(font
@@
 		)
 		(instances
-			(project "014_Sensor_PI_RS485 board"
+			(project "002_Sensor_PI_RS485 board"
 				(path "/b0089fb8-2318-4750-8145-7647caa10afa/8abbdb56-ea85-4864-aa21-196a08be6eef"
 					(page "28")
@@
 		)
 		(fill
-			(color 0 0 0 0.0000)
+			(color 0 0 0 0)
 		)
 		(property "Sheetname" "4_Sensor_bank4"
 			(at 74.93 36.1184 0)
+			(show_name no)
+			(do_not_autoplace no)
 			(effects
 				(font
@@
 		(property "Sheetfile" "4_Sensor_Bank.kicad_sch"
 			(at 74.93 57.7346 0)
+			(show_name no)
+			(do_not_autoplace no)
 			(effects
 				(font
@@
 		(property "Field2" ""
 			(at 74.93 36.83 0)
+			(show_name no)
+			(do_not_autoplace no)
 			(effects
 				(font
@@
 		)
 		(instances
-			(project "014_Sensor_PI_RS485 board"
+			(project "002_Sensor_PI_RS485 board"
 				(path "/b0089fb8-2318-4750-8145-7647caa10afa/8abbdb56-ea85-4864-aa21-196a08be6eef"
 					(page "23")
@@
 		)
 		(fill
-			(color 0 0 0 0.0000)
+			(color 0 0 0 0)
 		)
 		(property "Sheetname" "4_Sensor_bank1"
 			(at 21.59 64.0584 0)
+			(show_name no)
+			(do_not_autoplace no)
 			(effects
 				(font
@@
 		(property "Sheetfile" "4_Sensor_Bank.kicad_sch"
 			(at 21.59 85.6746 0)
+			(show_name no)
+			(do_not_autoplace no)
 			(effects
 				(font
@@
 		(property "Field2" ""
 			(at 21.59 64.77 0)
+			(show_name no)
+			(do_not_autoplace no)
 			(effects
 				(font
@@
 		)
 		(instances
-			(project "014_Sensor_PI_RS485 board"
+			(project "002_Sensor_PI_RS485 board"
 				(path "/b0089fb8-2318-4750-8145-7647caa10afa/8abbdb56-ea85-4864-aa21-196a08be6eef"
 					(page "8")
@@
 		)
 		(fill
-			(color 0 0 0 0.0000)
+			(color 0 0 0 0)
 		)
 		(property "Sheetname" "4_Sensor_bank3"
 			(at 21.59 119.9384 0)
+			(show_name no)
+			(do_not_autoplace no)
 			(effects
 				(font
@@
 		(property "Sheetfile" "4_Sensor_Bank.kicad_sch"
 			(at 21.59 141.5546 0)
+			(show_name no)
+			(do_not_autoplace no)
 			(effects
 				(font
@@
 		(property "Field2" ""
 			(at 21.59 120.65 0)
+			(show_name no)
+			(do_not_autoplace no)
 			(effects
 				(font
@@
 		)
 		(instances
-			(project "014_Sensor_PI_RS485 board"
+			(project "002_Sensor_PI_RS485 board"
 				(path "/b0089fb8-2318-4750-8145-7647caa10afa/8abbdb56-ea85-4864-aa21-196a08be6eef"
 					(page "18")
