File: hardware/kicad/002_sensor_board_example/last_sensor_bank.kicad_sch (KiCad schematic)
At the start: 6 parts, among them U3801 TLA2518IRTER

Commit message: Main Controller Board (1D) now added. Cheaper design, with RP2354, and BUCK PMIC
Other:
- company: (none) -> Noah Jaffe

Commit message: 001d bumped to 5V RS485 bus voltage. Sensor board schematic cleaned up, layout not begun
Parts:
- added C3804, C3805, C3806, C3807: 1 nF, Capacitor_SMD:C_0402_1005Metric, symbol Device:C
- added H3802, H3803: Mousebites to detatch sensor, custom_mousebite:mousebite, symbol Mechanical:MountingHole
- H3801: value Mousebites to detatch last sensor -> Mousebites to detatch sensor
Connections:
- net GND: now also C3804.2, C3805.2, C3806.2, C3807.2
- net Y0: now also C3804.1
- net Y1: now also C3805.1
- net Y2: now also C3806.1
- net Y3: now also C3807.1
Other:
- note added: "Place these caps next to ADC input pins"
- moved on the sheet: H3801
