File: hardware/kicad/002_sensor_board_example/last_sensor_bank.kicad_sch (KiCad schematic)
At the start: 12 parts, among them U3801 TLA2518IRTER

Commit message: 002 sensor board: 5V bus rework, library consolidation, DRC pass
Board (002):
- Remove SS14 bridging diode; USB-C VBUS and JST V+ are now one net.
  Worst case is back-powering a host's VBUS, acceptable in a uniform
  5V fleet, and it drops 185mW in the bridging case.
- Remove the 8x 47k CS pull-ups. At 47k they parked the TLA2518 CS
  inputs mid-rail (1.7-2.1V, between VIL 0.99 and VIH 2.31); the
  internal pull-down now defines them cleanly low. Firmware must drive
  CS high before configuring SPI.
- 5V pour along the bottom edge, 3.3V moved up to the mounting rail.
- USB-C relocated; ~200mm D+/D- run on F.Cu over the B.Cu GND pour.
- Screw-head keepouts on all mounting holes.
- Board grown 2mm in Y -> 413.66 x 35.00 mm.

Net classes:
- USB_DIFF_90 -> USB_FS, diff pair 0.8/0.15 -> 0.35/0.15. The old name
  claimed 90 ohm; on a 1.51mm 2-layer stackup it is ~140 ohm and cannot
  be otherwise. Irrelevant at Full Speed.
- Add PWR_5V (+5V) and RS485 (/RS485_P, /RS485_N).
- Restore the +3V3 -> VCC assignment lost during the rename.

Libraries:
- footprints/ -> footprints.pretty/ so KiCad will save into it.
- Consolidate symbols into PHOTON / PHOTON_Modified on 001d and 002;
  drop unused vendor-exported libraries.
- Add mousebite_34mm: 17x 1.2mm NPTH at 2mm pitch. 0.8mm webs cut more
  easily than the old 1.4mm and still pass a 0.3mm trace.
- Fix MountingHole_2.7mm_M2.5_Keepout: it disallowed pads, so each hole
  flagged its own NPTH (17 DRC errors).

Fab outputs now tracked via .gitignore negation for production/*.csv.

Co-Authored-By: Claude Opus 5 <noreply@anthropic.com>
Parts:
- removed R3801: 47k, Resistor_SMD:R_0402_1005Metric, symbol Device:R
- C3807: now not fitted; now left out of the parts list
- H3801, H3802, H3803: footprint custom_mousebite:mousebite -> footprints:mousebite_34mm
- U3801: symbol tla2518:TLA2518IRTER -> PHOTON:TLA2518IRTER
Changed lines of the file:
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@@
 		(color 0 0 0 0)
 	)
-	(junction
-		(at 187.96 118.11)
-		(diameter 0)
-		(color 0 0 0 0)
-	)
 	(wire
 		(pts
@@
 	(wire
 		(pts
-			(xy 190.5 118.11) (xy 187.96 118.11)
-		)
-		(stroke
-			(width 0)
-			(type default)
-		)
-	)
-	(wire
-		(pts
 			(xy 102.87 78.74) (xy 109.22 78.74)
 		)
@@
 	(wire
 		(pts
-			(xy 187.96 118.11) (xy 166.37 118.11)
+			(xy 166.37 118.11) (xy 190.5 118.11)
 		)
 		(stroke
@@
 			)
 		)
-		(property "Footprint" "custom_mousebite:mousebite"
+		(property "Footprint" "footprints:mousebite_34mm"
 			(at 144.78 69.85 0)
 			(hide yes)
@@
 	)
 	(symbol
-		(lib_id "power:VCC")
-		(at 187.96 110.49 0)
-		(unit 1)
-		(body_style 1)
-		(exclude_from_sim no)
-		(in_bom yes)
-		(on_board yes)
-		(in_pos_files yes)
-		(dnp no)
-		(property "Reference" "#PWR03801"
-			(at 187.96 114.3 0)
-			(hide yes)
-			(show_name no)
-			(do_not_autoplace no)
-			(effects
-				(font
-					(size 1.27 1.27)
-				)
-			)
-		)
-		(property "Value" "+3V3"
-			(at 186.436 106.426 0)
-			(show_name no)
-			(do_not_autoplace no)
-			(effects
-				(font
-					(size 1.27 1.27)
-				)
-			)
-		)
-		(property "Footprint" ""
-			(at 187.96 110.49 0)
-			(hide yes)
-			(show_name no)
-			(do_not_autoplace no)
-			(effects
-				(font
-					(size 1.27 1.27)
-				)
-			)
-		)
-		(property "Datasheet" ""
-			(at 187.96 110.49 0)
-			(hide yes)
-			(show_name no)
-			(do_not_autoplace no)
-			(effects
-				(font
-					(size 1.27 1.27)
-				)
-			)
-		)
-		(property "Description" "Power symbol creates a global label with name \"VCC\""
-			(at 187.96 110.49 0)
-			(hide yes)
-			(show_name no)
-			(do_not_autoplace no)
-			(effects
-				(font
-					(size 1.27 1.27)
-				)
-			)
-		)
-		(pin "1"
-		)
-		(instances
-			(project "002_Sensor_PI_RS485 board"
-				(path "/b0089fb8-2318-4750-8145-7647caa10afa/8abbdb56-ea85-4864-aa21-196a08be6eef/80523f9a-b0b8-4efa-b3d9-d2f9096ba0cd"
-					(reference "#PWR03801")
-					(unit 1)
-				)
-			)
-		)
-	)
-	(symbol
 		(lib_id "power:GND")
 		(at 180.34 102.87 0)
@@
 		(unit 1)
 		(body_style 1)
-		(exclude_from_sim no)
-		(in_bom yes)
-		(on_board yes)
-		(in_pos_files yes)
-		(dnp no)
+		(exclude_from_sim yes)
+		(in_bom no)
+		(on_board no)
+		(in_pos_files no)
+		(dnp yes)
 		(property "Reference" "C3807"
 			(at 255.016 112.522 0)
@@
 	)
 	(symbol
-		(lib_id "tla2518:TLA2518IRTER")
+		(lib_id "PHOTON:TLA2518IRTER")
 		(at 100.33 102.87 0)
 		(unit 1)
@@
 			)
 		)
-		(property "Footprint" "custom_mousebite:mousebite"
+		(property "Footprint" "footprints:mousebite_34mm"
 			(at 144.78 63.5 0)
 			(hide yes)
@@
 			)
 		)
-		(property "Footprint" "custom_mousebite:mousebite"
+		(property "Footprint" "footprints:mousebite_34mm"
 			(at 144.78 76.2 0)
 			(hide yes)
@@
 					(unit 1)
 				)
-			)
-		)
-	)
-	(symbol
-		(lib_id "Device:R")
-		(at 187.96 114.3 0)
-		(unit 1)
-		(body_style 1)
-		(exclude_from_sim no)
-		(in_bom yes)
-		(on_board yes)
-		(in_pos_files yes)
-		(dnp no)
-		(fields_autoplaced yes)
-		(property "Reference" "R3801"
-			(at 190.5 113.0299 0)
-			(show_name no)
-			(do_not_autoplace no)
-			(effects
-				(font
-					(size 1.27 1.27)
-				)
-				(justify left)
-			)
-		)
-		(property "Value" "47k"
-			(at 190.5 115.5699 0)
-			(show_name no)
-			(do_not_autoplace no)
-			(effects
-				(font
-					(size 1.27 1.27)
-				)
-				(justify left)
-			)
-		)
-		(property "Footprint" "Resistor_SMD:R_0402_1005Metric"
-			(at 186.182 114.3 90)
-			(hide yes)
-			(show_name no)
-			(do_not_autoplace no)
-			(effects
-				(font
-					(size 1.27 1.27)
-				)
-			)
-		)
-		(property "Datasheet" ""
-			(at 187.96 114.3 0)
-			(hide yes)
-			(show_name no)
-			(do_not_autoplace no)
-			(effects
-				(font
-					(size 1.27 1.27)
-				)
-			)
-		)
-		(property "Description" "Resistor"
-			(at 187.96 114.3 0)
-			(hide yes)
-			(show_name no)
-			(do_not_autoplace no)
-			(effects
-				(font
-					(size 1.27 1.27)
-				)
-			)
-		)
-		(pin "1"
-		)
-		(pin "2"
-		)
-		(instances
-			(project "002_Sensor_PI_RS485 board"
-				(path "/b0089fb8-2318-4750-8145-7647caa10afa/8abbdb56-ea85-4864-aa21-196a08be6eef/80523f9a-b0b8-4efa-b3d9-d2f9096ba0cd"
-					(reference "R3801")
-					(unit 1)
-				)

Commit message: 002: ERC/DRC to zero, symbol and value cleanup
Schematic (ERC 24 -> 0):
- VCNT2020 renamed to VCNT2025X01, matching the part actually fitted.
  Pin types preserved: passive / open_collector / passive / passive.
  The old auto-generated VCNT2025X01 symbol (all pins Unspecified) is gone.
- THVD1424RGTR: 10 pins off Unspecified (R, RE, DE, D, TERM_TX, TERM_RX,
  Y, Z, VIO, H/F). VIO was typed as a signal despite being a supply pin.
- TLA2518IRTER: DECAP -> Passive, clearing 8 warnings at once.
- PWR_FLAG moved off J3's VBUS (which J3 already drives as a Power output)
  onto GND, which had none. One move, two errors.
- JP1/JP2/JP4 repointed to stock Jumper:SolderJumper_2_Open. The project
  copy was KiCad's older stock symbol, not a deliberate modification.
- R1 1M -> 0 ohm, bonding the USB-C shell to GND. A lone 1M is a static
  bleed, not a shield connection: open at every frequency that matters,
  and it isolated nothing since J3's GND pins are already bonded.

Layout:
- MountingHole keepout had (pads not_allowed), so each hole flagged its
  own NPTH. Fixed and patched into all 17 instances.
- Mousebite silkscreen removed (library + all 3 placements). The dashed
  line crossed the pours end to end and caused ~61 of the DRC warnings.
- 30 duplicate vias deleted. Each pair was 1 nm apart from a float->int
  round-trip in the layout plugin, so KiCad's "delete redundant vias"
  could not see them while DRC's co-located check could.
- min_resolved_spokes 2 -> 1; single-spoke pads are accepted on this
  board rather than excluded per-violation.

BOM hygiene:
- Component values normalised: no space before units, ASCII u instead of
  U+03BC, and 3.3u given its missing unit. Merges 100 kohm/100kohm and
  1 uF/1uF, which would otherwise export as separate lines for identical
  parts. 181 edits across schematics and PCB, kept in sync.

Libraries:
- PHOTON_Modified reduced to the two symbols that genuinely diverge from
  stock: Crystal_GND24 and USB_C_Receptacle_USB2.0.

Known o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
Parts:
- C3801, C3802, C3803: value 1 uF -> 1uF
- C3804, C3805, C3806, C3807: value 1 nF -> 1nF
- U3801: JLCPCB Part # (none) -> C1855741
Changed lines of the file:
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@@
 			)
 		)
-		(property "Value" "1 uF"
+		(property "Value" "1uF"
 			(at 82.042 124.206 0)
 			(show_name no)
@@
 			)
 		)
-		(property "Value" "1 uF"
+		(property "Value" "1uF"
 			(at 172.212 134.366 0)
 			(show_name no)
@@
 			)
 		)
-		(property "Value" "1 nF"
+		(property "Value" "1nF"
 			(at 241.808 116.078 0)
 			(show_name no)
@@
 			)
 		)
-		(property "Value" "1 nF"
+		(property "Value" "1nF"
 			(at 213.868 116.078 0)
 			(show_name no)
@@
 			)
 		)
-		(property "Value" "1 uF"
+		(property "Value" "1uF"
 			(at 93.472 126.746 0)
 			(show_name no)
@@
 			)
 		)
-		(property "Value" "1 nF"
+		(property "Value" "1nF"
 			(at 227.838 116.078 0)
 			(show_name no)
@@
 			)
 		)
-		(property "Value" "1 nF"
+		(property "Value" "1nF"
 			(at 254.508 116.078 0)
 			(show_name no)
@@
 			(at 100.33 102.87 0)
 			(hide yes)
+			(show_name no)
+			(do_not_autoplace no)
+			(effects
+				(font
+					(size 1.27 1.27)
+				)
+			)
+		)
+		(property "JLCPCB Part #" "C1855741"
+			(at 100.33 102.87 0)
+			(hide yes)
