File: hardware/kicad/002_sensor_board_example/002_Sensor_PI_RS485 board.kicad_pcb (KiCad board)
At the start: 2 copper layers, 407.6 x 25 mm, 276 parts, among them J1 JST_SH, J2 JST_SH, J3 USB_C_Receptacle_USB2.0, Q1001 AO3400A, Q1101 AO3400A, Q1201 AO3400A, Q1401 AO3400A, Q1501 AO3400A, Q1601 AO3400A, Q1701 AO3400A, Q1901 AO3400A, Q2001 AO3400A, Q2101 AO3400A, Q2201 AO3400A, Q2401 AO3400A, Q2501 AO3400A, Q2601 AO3400A, Q2701 AO3400A, Q2901 AO3400A, Q3001 AO3400A, Q301 AO3400A, Q3101 AO3400A, Q3201 AO3400A, Q3401 AO3400A, Q3501 AO3400A, Q3601 AO3400A, Q3701 AO3400A, Q4301 AO3400A, Q4401 AO3400A, Q4501 AO3400A, Q501 AO3400A, Q601 AO3400A, Q701 AO3400A, Q901 AO3400A, SW1 SW_SPST, SW2 SW_SPST, U1 RP2350_60QFN, U1001 VCNT2025X01, U1101 VCNT2025X01, U1201 VCNT2025X01, U1301 TLA2518IRTER, U1401 VCNT2025X01, U1501 VCNT2025X01, U1601 VCNT2025X01, U1701 VCNT2025X01, U1801 TLA2518IRTER, U1901 VCNT2025X01, U2 NCP1117-3.3_SOT223, U2001 VCNT2025X01, U2101 VCNT2025X01, U2201 VCNT2025X01, U2301 TLA2518IRTER, U2401 VCNT2025X01, U2501 VCNT2025X01, U2601 VCNT2025X01, U2701 VCNT2025X01, U2801 TLA2518IRTER, U2901 VCNT2025X01, U3 W25Q128JVPIQ, U3001 VCNT2025X01, U301 VCNT2025X01, U3101 VCNT2025X01, U3201 VCNT2025X01, U3301 TLA2518IRTER, U3401 VCNT2025X01, U3501 VCNT2025X01, U3601 VCNT2025X01, U3701 VCNT2025X01, U3801 TLA2518IRTER, U4 TPD4E05U06DQAR, U401 TLA2518IRTER, U4301 VCNT2025X01, U4401 VCNT2025X01, U4501 VCNT2025X01, U5 THVD1424RGTR, U501 VCNT2025X01, U601 VCNT2025X01, U701 VCNT2025X01, U801 TLA2518IRTER, U901 VCNT2025X01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

Commit message: 002 sensor board: 5V bus rework, library consolidation, DRC pass
Board (002):
- Remove SS14 bridging diode; USB-C VBUS and JST V+ are now one net.
  Worst case is back-powering a host's VBUS, acceptable in a uniform
  5V fleet, and it drops 185mW in the bridging case.
- Remove the 8x 47k CS pull-ups. At 47k they parked the TLA2518 CS
  inputs mid-rail (1.7-2.1V, between VIL 0.99 and VIH 2.31); the
  internal pull-down now defines them cleanly low. Firmware must drive
  CS high before configuring SPI.
- 5V pour along the bottom edge, 3.3V moved up to the mounting rail.
- USB-C relocated; ~200mm D+/D- run on F.Cu over the B.Cu GND pour.
- Screw-head keepouts on all mounting holes.
- Board grown 2mm in Y -> 413.66 x 35.00 mm.

Net classes:
- USB_DIFF_90 -> USB_FS, diff pair 0.8/0.15 -> 0.35/0.15. The old name
  claimed 90 ohm; on a 1.51mm 2-layer stackup it is ~140 ohm and cannot
  be otherwise. Irrelevant at Full Speed.
- Add PWR_5V (+5V) and RS485 (/RS485_P, /RS485_N).
- Restore the +3V3 -> VCC assignment lost during the rename.

Libraries:
- footprints/ -> footprints.pretty/ so KiCad will save into it.
- Consolidate symbols into PHOTON / PHOTON_Modified on 001d and 002;
  drop unused vendor-exported libraries.
- Add mousebite_34mm: 17x 1.2mm NPTH at 2mm pitch. 0.8mm webs cut more
  easily than the old 1.4mm and still pass a 0.3mm trace.
- Fix MountingHole_2.7mm_M2.5_Keepout: it disallowed pads, so each hole
  flagged its own NPTH (17 DRC errors).

Fab outputs now tracked via .gitignore negation for production/*.csv.

Co-Authored-By: Claude Opus 5 <noreply@anthropic.com>
Parts:
- removed CR2: PTVSHC3D7VU, footprints:SOD-323_L1.8-W1.3-LS2.5-RD
- removed J4: ~, Connector_PinHeader_1.27mm:PinHeader_1x04_P1.27mm_Vertical
- removed R17: 100kΩ, Resistor_SMD:R_0402_1005Metric
- removed the R4 at (370.5, 18.9)
- removed SW1, SW2: SW_SPST, footprints:SW-TH_MSK12C02
- removed U2: NCP1117-3.3_SOT223, Package_TO_SOT_SMD:SOT-223-3_TabPin2
- removed U3: W25Q128JVPIQ, footprints:WSON_128JVPIQ_WIN
- added C23: 100nF, Capacitor_SMD:C_0402_1005Metric, F.Cu at (61.5, 24.2)
- added C24: 100nF, Capacitor_SMD:C_0402_1005Metric, F.Cu at (127.2, 23.2)
- added C25: 100nF, Capacitor_SMD:C_0402_1005Metric, F.Cu at (323.8, 23.9)
- added C26: 100nF, Capacitor_SMD:C_0402_1005Metric, F.Cu at (260.1, 23.3)
- added C27: 100nF, Capacitor_SMD:C_0402_1005Metric, F.Cu at (210.3, 23.9)
- added C3804: 1 nF, Capacitor_SMD:C_0402_1005Metric, F.Cu at (364.2, 8.78)
- added C3805: 1 nF, Capacitor_SMD:C_0402_1005Metric, F.Cu at (366.1, 11.1)
- added C3806: 1 nF, Capacitor_SMD:C_0402_1005Metric, F.Cu at (366.1, 13.8)
- added H10: MountingHole, footprints:MountingHole_2.7mm_M2.5_Keepout, F.Cu at (402.4, -4.00)
- added H11: MountingHole, footprints:MountingHole_2.7mm_M2.5_Keepout, F.Cu at (389.5, -4.00)
- added H12: MountingHole, footprints:MountingHole_2.7mm_M2.5_Keepout, F.Cu at (378.8, 22.8)
- added H13: MountingHole, footprints:MountingHole_2.7mm_M2.5_Keepout, F.Cu at (50.0, 22.8)
- added H14: MountingHole, footprints:MountingHole_2.7mm_M2.5_Keepout, F.Cu at (248.4, 22.8)
- added H15: MountingHole, footprints:MountingHole_2.7mm_M2.5_Keepout, F.Cu at (106.5, 22.8)
- added H16: MountingHole, footprints:MountingHole_2.7mm_M2.5_Keepout, F.Cu at (378.3, -4.00)
- added H17: MountingHole, footprints:MountingHole_2.7mm_M2.5_Keepout, F.Cu at (312.4, 22.8)
- added H3802: Mousebites to detatch sensor, footprints:mousebite_34mm, F.Cu at (371.6, 9.60)
- added H3803: Mousebites to detatch sensor, footprints:mousebite_34mm, F.Cu at (384.0, 9.60)
- added H5: MountingHole, footprints:MountingHole_2.7mm_M2.5_Keepout, F.Cu at (88.9, -4.00)
- added H6: MountingHole, footprints:MountingHole_2.7mm_M2.5_Keepout, F.Cu at (155.2, -4.00)
- added H7: MountingHole, footprints:MountingHole_2.7mm_M2.5_Keepout, F.Cu at (221.7, -4.00)
- added H8: MountingHole, footprints:MountingHole_2.7mm_M2.5_Keepout, F.Cu at (289.1, -4.00)
- added H9: MountingHole, footprints:MountingHole_2.7mm_M2.5_Keepout, F.Cu at (350.2, -4.00)
- added JP1: SolderJumper_2_Open, Jumper:SolderJumper-2_P1.3mm_Open_RoundedPad1.0x1.5mm, F.Cu at (38.9, 20.1)
- added L2: 1 uH, Inductor_SMD:L_1008_2520Metric, F.Cu at (14.9, 19.9)
- added R103: 100kΩ, Resistor_SMD:R_0402_1005Metric, F.Cu at (12.8, 15.8)
- added R104: 300kΩ, Resistor_SMD:R_0402_1005Metric, F.Cu at (12.8, 13.8)
- added R105: 150kΩ, Resistor_SMD:R_0402_1005Metric, F.Cu at (12.8, 14.8)
- added R5: 120 Ω, Resistor_SMD:R_0402_1005Metric, F.Cu at (358.8, 21.2)
- added U6: TPS62A0569ADRLR, footprints:SOT-563_DRL0006A, F.Cu at (13.1, 17.4)
- C1: value 10uF -> 4.7uF
- C4: value 10uF -> 22uF
- H1, H2, H3, H4: footprint MountingHole:MountingHole_2.7mm_M2.5 -> footprints:MountingHole_2.7mm_M2.5_Keepout
- H3801: value Mousebites to detatch last sensor -> Mousebites to detatch sensor; footprint custom_mousebite:mousebite -> footprints:mousebite_34mm
- JP2: value SolderJumper_2_Bridged -> SolderJumper_2_Open; footprint Jumper:SolderJumper-2_P1.3mm_Bridged_RoundedPad1.0x1.5mm -> Jumper:SolderJumper-2_P1.3mm_Open_RoundedPad1.0x1.5mm
- U1: value RP2350_60QFN -> RP2354_60QFN
- moved C4 260.8 mm to (15.9, 16.8), turned to 90 degrees
- moved H4 252.4 mm to (10.3, -4.00)
- moved R1 250.7 mm to (5.30, 11.8), turned to 180 degrees
- moved CR1 250.5 mm to (7.25, 16.0), turned to 90 degrees
- moved J3 250.3 mm to (-1.25, 19.2), turned to -90 degrees
- moved C1 250.0 mm to (10.8, 17.1), turned to 90 degrees
- moved R2 246.6 mm to (5.13, 21.8), turned to 180 degrees
- moved FB1 246.4 mm to (11.4, 19.6)
- moved U4 244.3 mm to (5.03, 19.4), turned to 180 degrees
- moved R3 243.8 mm to (6.88, 21.3), turned to 90 degrees
- moved C22 200.5 mm to (14.2, 24.6), turned to 0 degrees
- moved JP2 92.3 mm to (355.9, 20.9), turned to 180 degrees
- moved J1 24.5 mm to (33.0, 20.8)
- moved C3801 18.7 mm to (361.4, 9.21)
- moved C3802 18.7 mm to (361.4, 10.3)
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- renumbered JP101 to JP4, R101 to R4
Connections:
- net /FLASH_SS renamed /QSPI_SS
- C1 pad 1: Net-(JP2-A) -> Net-(U6-EN)
- C22 pad 1: +3V3 -> +5V
- CR1 pad 1: VBUS -> +5V
- FB1 pad 1: VBUS -> +5V
- FB1 pad 2: Net-(JP2-A) -> Net-(U6-EN)
- J1 pad 2: +3V3 -> +5V
- J2 pad 2: +3V3 -> +5V
- J3 pad A4: VBUS -> +5V
- J3 pad A9: VBUS -> +5V
- J3 pad B4: VBUS -> +5V
- J3 pad B9: VBUS -> +5V
- JP2 pad 1: Net-(JP2-A) -> /RS485_P
- R4 pad 2: /RS485_P -> /RS485_N
Routing:
- net /USB_D+: track 56.5 -> 225.5 mm
- net /USB_D-: track 57.7 -> 225.2 mm
- net /Sensor Array/Last_sensor_bank/EN2: track 20.7 -> 51.0 mm
- net +5V: track 0.00 -> 25.9 mm, vias 0 -> 8
- net /Sensor Array/4_Sensor_bank6/EN3: track 30.3 -> 4.96 mm
- net /Sensor Array/Last_sensor_bank/Y2: track 25.8 -> 51.0 mm
- net /Sensor Array/Last_sensor_bank/EN1: track 7.09 -> 32.1 mm
- net /GPIO0: track 211.6 -> 187.4 mm, vias 4 -> 2
- net /Sensor Array/Last_sensor_bank/Y1: track 11.3 -> 33.7 mm
- net /UART_TX: track 28.0 -> 50.2 mm
- net VBUS: track 21.2 -> 0.00 mm
- net /GPIO3: track 218.9 -> 200.3 mm, vias 12 -> 10
- net /SPI1_SCLK: track 207.8 -> 189.8 mm, vias 10 -> 8
- net /BANK_7_CS: track 197.4 -> 180.4 mm, vias 6 -> 4
- net /RS485_N: track 391.3 -> 374.6 mm, vias 8 -> 2
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- added copper zone on F.Cu, net +5V
Other:
- board size 407.6 x 25 mm -> 413.7 x 35 mm
- board text added: "USB Boot"
- board text added: "klavecimbel.com RP2354 Sensor Board A007 REV B github.com/w4iei/photon"
- board text removed: "LDO Disable"
- board text removed: "Noah Jaffe RP2350 Sensor Board A007 REV A github.com/w4iei/photon"
- board text removed: "RS-485 TERM OFF ON"
- board text removed: "Short for USB Boot"
