File: hardware/kicad/002_sensor_board_example/002_Sensor_PI_RS485 board.kicad_pcb (KiCad board)
At the start: 2 copper layers, 413.7 x 35 mm, 298 parts, among them J1 JST_SH, J2 JST_SH, J3 USB_C_Receptacle_USB2.0, Q1001 AO3400A, Q1101 AO3400A, Q1201 AO3400A, Q1401 AO3400A, Q1501 AO3400A, Q1601 AO3400A, Q1701 AO3400A, Q1901 AO3400A, Q2001 AO3400A, Q2101 AO3400A, Q2201 AO3400A, Q2401 AO3400A, Q2501 AO3400A, Q2601 AO3400A, Q2701 AO3400A, Q2901 AO3400A, Q3001 AO3400A, Q301 AO3400A, Q3101 AO3400A, Q3201 AO3400A, Q3401 AO3400A, Q3501 AO3400A, Q3601 AO3400A, Q3701 AO3400A, Q4301 AO3400A, Q4401 AO3400A, Q4501 AO3400A, Q501 AO3400A, Q601 AO3400A, Q701 AO3400A, Q901 AO3400A, U1 RP2354_60QFN, U1001 VCNT2025X01, U1101 VCNT2025X01, U1201 VCNT2025X01, U1301 TLA2518IRTER, U1401 VCNT2025X01, U1501 VCNT2025X01, U1601 VCNT2025X01, U1701 VCNT2025X01, U1801 TLA2518IRTER, U1901 VCNT2025X01, U2001 VCNT2025X01, U2101 VCNT2025X01, U2201 VCNT2025X01, U2301 TLA2518IRTER, U2401 VCNT2025X01, U2501 VCNT2025X01, U2601 VCNT2025X01, U2701 VCNT2025X01, U2801 TLA2518IRTER, U2901 VCNT2025X01, U3001 VCNT2025X01, U301 VCNT2025X01, U3101 VCNT2025X01, U3201 VCNT2025X01, U3301 TLA2518IRTER, U3401 VCNT2025X01, U3501 VCNT2025X01, U3601 VCNT2025X01, U3701 VCNT2025X01, U3801 TLA2518IRTER, U4 TPD4E05U06DQAR, U401 TLA2518IRTER, U4301 VCNT2025X01, U4401 VCNT2025X01, U4501 VCNT2025X01, U5 THVD1424RGTR, U501 VCNT2025X01, U6 TPS62A0569ADRLR, U601 VCNT2025X01, U701 VCNT2025X01, U801 TLA2518IRTER, U901 VCNT2025X01, Y1 ABM8-272-T3

Commit message: 002: ERC/DRC to zero, symbol and value cleanup
Schematic (ERC 24 -> 0):
- VCNT2020 renamed to VCNT2025X01, matching the part actually fitted.
  Pin types preserved: passive / open_collector / passive / passive.
  The old auto-generated VCNT2025X01 symbol (all pins Unspecified) is gone.
- THVD1424RGTR: 10 pins off Unspecified (R, RE, DE, D, TERM_TX, TERM_RX,
  Y, Z, VIO, H/F). VIO was typed as a signal despite being a supply pin.
- TLA2518IRTER: DECAP -> Passive, clearing 8 warnings at once.
- PWR_FLAG moved off J3's VBUS (which J3 already drives as a Power output)
  onto GND, which had none. One move, two errors.
- JP1/JP2/JP4 repointed to stock Jumper:SolderJumper_2_Open. The project
  copy was KiCad's older stock symbol, not a deliberate modification.
- R1 1M -> 0 ohm, bonding the USB-C shell to GND. A lone 1M is a static
  bleed, not a shield connection: open at every frequency that matters,
  and it isolated nothing since J3's GND pins are already bonded.

Layout:
- MountingHole keepout had (pads not_allowed), so each hole flagged its
  own NPTH. Fixed and patched into all 17 instances.
- Mousebite silkscreen removed (library + all 3 placements). The dashed
  line crossed the pours end to end and caused ~61 of the DRC warnings.
- 30 duplicate vias deleted. Each pair was 1 nm apart from a float->int
  round-trip in the layout plugin, so KiCad's "delete redundant vias"
  could not see them while DRC's co-located check could.
- min_resolved_spokes 2 -> 1; single-spoke pads are accepted on this
  board rather than excluded per-violation.

BOM hygiene:
- Component values normalised: no space before units, ASCII u instead of
  U+03BC, and 3.3u given its missing unit. Merges 100 kohm/100kohm and
  1 uF/1uF, which would otherwise export as separate lines for identical
  parts. 181 edits across schematics and PCB, kept in sync.

Libraries:
- PHOTON_Modified reduced to the two symbols that genuinely diverge from
  stock: Crystal_GND24 and USB_C_Receptacle_USB2.0.

Known o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
Parts:
- added H18: MountingHole, footprints:MountingHole_2.7mm_M2.5_Keepout, F.Cu at (365.0, 22.8)
- C10: value 1μF -> 1uF
- C1301, C1302, C1303, C1801, C1802, C1803, C2301, C2302, C2303, C2801, C2802, C2803, C3301, C3302, C3303, C3801, C3802, C3803, C401, C402, C403, C801, C802, C803: value 1 uF -> 1uF
- C1304, C1305, C1306, C1307, C1804, C1805, C1806, C1807, C2304, C2305, C2306, C2307, C2804, C2805, C2806, C2807, C3304, C3305, C3306, C3307, C3804, C3805, C3806, C404, C405, C406, C407, C804, C805, C806, C807: value 1 nF -> 1nF
- L1: value 3.3u -> 3.3uH
- L2: value 1 uH -> 1uH
- R1: value 1MΩ -> 0Ω; footprint Resistor_SMD:R_0805_2012Metric_Pad1.20x1.40mm_HandSolder -> Resistor_SMD:R_0402_1005Metric
- R1001, R1101, R1201, R1401, R1501, R1601, R1701, R1901, R2001, R2101, R2201, R2401, R2501, R2601, R2701, R2901, R3001, R301, R3101, R3201, R3401, R3501, R3601, R3701, R4301, R4401, R4501, R501, R601, R701, R901: value 100 kΩ -> 100kΩ
- R1002, R1102, R1202, R1402, R1502, R1602, R1702, R1902, R2002, R2102, R2202, R2402, R2502, R2602, R2702, R2902, R3002, R302, R3102, R3202, R3402, R3502, R3602, R3702, R4302, R4402, R4502, R502, R602, R702, R902: value 68 Ω -> 68Ω
- R1003, R1103, R1203, R1403, R1503, R1603, R1703, R1903, R2003, R2103, R2203, R2403, R2503, R2603, R2703, R2903, R3003, R303, R3103, R3203, R3403, R3503, R3603, R3703, R4303, R4403, R4503, R503, R603, R703, R903: value 4.7 kΩ -> 4.7kΩ
- R2, R3: value 5.1 kΩ -> 5.1kΩ
- R4, R5: value 120 Ω -> 120Ω
- moved J2 16.2 mm to (348.3, 22.8)
- moved JP2 16.2 mm to (339.6, 20.8)
- moved R5 16.2 mm to (342.5, 21.1)
- moved R1 2.96 mm to (2.58, 13.0), turned to 0 degrees
- moved R2703 0.71 mm to (253.6, 2.92), turned to 0 degrees
- moved R2103 0.65 mm to (187.1, 2.90), turned to 0 degrees
- moved C21 0.64 mm to (197.5, 9.87), turned to 135 degrees
- moved R2203 0.62 mm to (200.4, 2.92), turned to 0 degrees
- moved J3 0.60 mm to (-1.84, 19.2)
- moved R13 0.23 mm to (200.8, 8.40)
Connections:
- R1 pad 1: GND -> Net-(J3-SHIELD)
- R1 pad 2: Net-(J3-SHIELD) -> GND
Routing:
- net /RS485_N: track 374.6 -> 358.5 mm
- net /RS485_P: track 373.4 -> 357.4 mm
- net +3V3: track 112.7 -> 105.6 mm, vias 10 -> 8
- net /Sensor Array/4_Sensor_bank6/EN3: track 4.96 -> 11.0 mm
- net Net-(J3-SHIELD): track 4.27 -> 2.20 mm
- net /GPIO8: track 216.9 -> 214.9 mm
- net /BANK_3_CS: track 26.5 -> 24.6 mm
- net /GPIO11: track 210.1 -> 208.5 mm
- net /SPI0_SCLK: track 208.0 -> 206.9 mm
- net GND: track 308.3 -> 308.5 mm, vias 220 -> 192
Other:
- outline, holes or cut-outs redrawn
- board text added: "Noah Jaffe PHOTON Sensor Board A007 REV B github.com/w4iei/photon"
- board text removed: "klavecimbel.com RP2354 Sensor Board A007 REV B github.com/w4iei/photon"
