File: hardware/kicad/002_sensor_board/002_Sensor_PI_RS485 board.kicad_pcb (KiCad board)
At the start: 2 copper layers, 413.7 x 35 mm, 299 parts, among them J1 JST_SH, J2 JST_SH, J3 USB_C_Receptacle_USB2.0, Q1001 AO3400A, Q1101 AO3400A, Q1201 AO3400A, Q1401 AO3400A, Q1501 AO3400A, Q1601 AO3400A, Q1701 AO3400A, Q1901 AO3400A, Q2001 AO3400A, Q2101 AO3400A, Q2201 AO3400A, Q2401 AO3400A, Q2501 AO3400A, Q2601 AO3400A, Q2701 AO3400A, Q2901 AO3400A, Q3001 AO3400A, Q301 AO3400A, Q3101 AO3400A, Q3201 AO3400A, Q3401 AO3400A, Q3501 AO3400A, Q3601 AO3400A, Q3701 AO3400A, Q4301 AO3400A, Q4401 AO3400A, Q4501 AO3400A, Q501 AO3400A, Q601 AO3400A, Q701 AO3400A, Q901 AO3400A, U1 RP2354_60QFN, U1001 VCNT2025X01, U1101 VCNT2025X01, U1201 VCNT2025X01, U1301 TLA2518IRTER, U1401 VCNT2025X01, U1501 VCNT2025X01, U1601 VCNT2025X01, U1701 VCNT2025X01, U1801 TLA2518IRTER, U1901 VCNT2025X01, U2001 VCNT2025X01, U2101 VCNT2025X01, U2201 VCNT2025X01, U2301 TLA2518IRTER, U2401 VCNT2025X01, U2501 VCNT2025X01, U2601 VCNT2025X01, U2701 VCNT2025X01, U2801 TLA2518IRTER, U2901 VCNT2025X01, U3001 VCNT2025X01, U301 VCNT2025X01, U3101 VCNT2025X01, U3201 VCNT2025X01, U3301 TLA2518IRTER, U3401 VCNT2025X01, U3501 VCNT2025X01, U3601 VCNT2025X01, U3701 VCNT2025X01, U3801 TLA2518IRTER, U4 TPD4E05U06DQAR, U401 TLA2518IRTER, U4301 VCNT2025X01, U4401 VCNT2025X01, U4501 VCNT2025X01, U5 THVD1424RGTR, U501 VCNT2025X01, U6 TPS62A0569ADRLR, U601 VCNT2025X01, U701 VCNT2025X01, U801 TLA2518IRTER, U901 VCNT2025X01, Y1 ABM8-272-T3

Commit message: 002 sensor board: Rev B ordered; rename folder, add schematic PDF
Board is at zero ERC and zero DRC and has shipped to fab as Rev B
(RS-485, 5 V bus). This commit captures exactly what was ordered.

- Rename 002_sensor_board_example -> 002_sensor_board. It stopped being
  an example some time ago.
- Add Schematic_revB.pdf.
- Replace the Rev A production outputs with the Rev B set actually sent:
  gerbers/drill zip, BOM, positions, designators, IPC netlist.

The BOM now carries LCSC part numbers for every specialty part, which
none of the previous exports did - VCNT2025X01 (C7431257) and
THVD1424RGTR (C5359161) in particular had only ever been matched in
JLC's web UI at order time, so they survived in neither the design, the
exports, nor 34 KiCad backups. Recorded in the schematic this time.

Values were normalised earlier today (no space before units, ASCII u,
3.3u given its missing unit), which merged 100 kohm/100kohm and
1 uF/1uF into single BOM lines.

Excluded: production_rev B.zip, a Finder-created archive of the
production folder carrying __MACOSX resource forks and a .DS_Store. The
real fab deliverable is production/*.zip.

Co-Authored-By: Claude Opus 5 <noreply@anthropic.com>
Parts:
- added R106: 51kΩ, Resistor_SMD:R_0402_1005Metric, F.Cu at (12.8, 14.8)
- D3: value LED GREEN -> LED RED; footprint LED_SMD:LED_0402_1005Metric -> LED_SMD:LED_0603_1608Metric
- R104: value 300kΩ -> 200kΩ
- R105: value 150kΩ -> 200kΩ
- moved C27 24.4 mm to (186.0, 22.0)
- moved C24 23.1 mm to (150.3, 21.1), turned to 180 degrees
- moved C17 3.18 mm to (192.6, 10.2)
- moved C18 3.18 mm to (192.5, 12.5)
- moved R18 3.18 mm to (193.6, 11.5)
- moved Y1 3.18 mm to (189.6, 11.3)
- moved C13 1.10 mm to (204.9, 16.9), turned to 45 degrees
- moved R11 1.06 mm to (206.5, 18.8)
- moved R12 1.06 mm to (205.8, 19.5)
- moved R104 1.04 mm to (12.8, 12.8)
- moved R105 1.02 mm to (12.8, 13.8)
- moved R8 0.55 mm to (53.1, 8.52)
- moved L1 0.39 mm to (203.9, 21.1)
Connections:
- R104 pad 1: +3V3 -> Net-(R104-Pad1)
- R104 pad 2: Net-(R104-Pad2) -> +3V3
- R105 pad 1: Net-(R104-Pad2) -> Net-(R105-Pad1)
- R105 pad 2: Net-(U6-FB) -> Net-(R104-Pad1)
Routing:
- net +3V3: track 105.6 -> 96.4 mm
- net /XOUT: track 9.38 -> 5.67 mm
- net /XIN: track 14.8 -> 11.3 mm
- net /SPI0_SCLK: track 206.9 -> 208.1 mm
- net /GPIO11: track 208.5 -> 209.6 mm
- net /QSPI_SD0: track 1.16 -> 0.00 mm
- net /USB_D+: track 225.5 -> 226.7 mm
- net /USB_D-: track 225.2 -> 226.4 mm
- net /BANK_3_CS: track 24.6 -> 25.7 mm
- net Net-(R105-Pad1): track 0.00 -> 1.01 mm
- net Net-(R104-Pad1): track 0.00 -> 1.00 mm
- net Net-(R104-Pad2): track 1.00 -> 0.00 mm
- net /GPIO8: track 214.9 -> 215.8 mm
- net /QSPI_SD1: track 0.85 -> 0.00 mm
- net GND: track 308.5 -> 307.9 mm, vias 192 -> 196
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