File: hardware/kicad/002_sensor_board/002_Sensor_PI_RS485 board.kicad_pcb (KiCad board)
At the start: 2 copper layers, 413.7 x 35 mm, 300 parts, among them J1 JST_SH, J2 JST_SH, J3 USB_C_Receptacle_USB2.0, Q1001 AO3400A, Q1101 AO3400A, Q1201 AO3400A, Q1401 AO3400A, Q1501 AO3400A, Q1601 AO3400A, Q1701 AO3400A, Q1901 AO3400A, Q2001 AO3400A, Q2101 AO3400A, Q2201 AO3400A, Q2401 AO3400A, Q2501 AO3400A, Q2601 AO3400A, Q2701 AO3400A, Q2901 AO3400A, Q3001 AO3400A, Q301 AO3400A, Q3101 AO3400A, Q3201 AO3400A, Q3401 AO3400A, Q3501 AO3400A, Q3601 AO3400A, Q3701 AO3400A, Q4301 AO3400A, Q4401 AO3400A, Q4501 AO3400A, Q501 AO3400A, Q601 AO3400A, Q701 AO3400A, Q901 AO3400A, U1 RP2354_60QFN, U1001 VCNT2025X01, U1101 VCNT2025X01, U1201 VCNT2025X01, U1301 TLA2518IRTER, U1401 VCNT2025X01, U1501 VCNT2025X01, U1601 VCNT2025X01, U1701 VCNT2025X01, U1801 TLA2518IRTER, U1901 VCNT2025X01, U2001 VCNT2025X01, U2101 VCNT2025X01, U2201 VCNT2025X01, U2301 TLA2518IRTER, U2401 VCNT2025X01, U2501 VCNT2025X01, U2601 VCNT2025X01, U2701 VCNT2025X01, U2801 TLA2518IRTER, U2901 VCNT2025X01, U3001 VCNT2025X01, U301 VCNT2025X01, U3101 VCNT2025X01, U3201 VCNT2025X01, U3301 TLA2518IRTER, U3401 VCNT2025X01, U3501 VCNT2025X01, U3601 VCNT2025X01, U3701 VCNT2025X01, U3801 TLA2518IRTER, U4 TPD4E05U06DQAR, U401 TLA2518IRTER, U4301 VCNT2025X01, U4401 VCNT2025X01, U4501 VCNT2025X01, U5 THVD1424RGTR, U501 VCNT2025X01, U6 TPS62A0569ADRLR, U601 VCNT2025X01, U701 VCNT2025X01, U801 TLA2518IRTER, U901 VCNT2025X01, Y1 ABM8-272-T3

Commit message: Consolidate footprints into a single shared library
All three boards carried their own copies of the same footprints - 79
files across 11 project libraries for 37 distinct footprints. Several
existed three times over (RP2350-QFN-60 ThermalVias, edge_holes,
TO-236_VIS-L, SON_NT2020_VIS, L_pol_2016, USB_Micro-B). Three copies
drift, and this project has already been bitten twice by a library and
a board disagreeing.

- New hardware/kicad/common.pretty holds all 37, verified byte-identical
  where they were duplicated: zero name collisions with differing
  content, so nothing had to be reconciled.
- Each board's fp-lib-table is now a single "common" entry. Previously
  001 alone had eight, and the nickname "footprints" meant a different
  library on each of the three boards - so lib_ids were rewritten per
  board, not globally.
- 459 footprint references across the three boards now resolve. That
  includes SparkFun-Qwiic:qwiic_8mm on 001, which was referenced but
  had never been in any fp-lib-table - broken before this change.

Also shrinks docs/images/reflective_sensor.png from 2816x1536 / 4.43 MB
to 1600x873 / 1.72 MB.

Co-Authored-By: Claude Opus 5 <noreply@anthropic.com>
Parts:
- C2, C3: footprint footprints:C_0402_1005Metric_small_pads -> common:C_0402_1005Metric_small_pads
- CR1: footprint footprints:SOD-323_L1.8-W1.3-LS2.5-RD -> common:SOD-323_L1.8-W1.3-LS2.5-RD
- H1, H10, H11, H12, H13, H14, H15, H16, H17, H18, H2, H3, H4, H5, H6, H7, H8, H9: footprint footprints:MountingHole_2.7mm_M2.5_Keepout -> common:MountingHole_2.7mm_M2.5_Keepout
- H3801, H3802, H3803: footprint footprints:mousebite_34mm -> common:mousebite_34mm
- L1: footprint footprints:L_pol_2016 -> common:L_pol_2016
- U1: footprint footprints:RP2350-QFN-60-1EP_7x7_P0.4mm_EP3.4x3.4mm_ThermalVias -> common:RP2350-QFN-60-1EP_7x7_P0.4mm_EP3.4x3.4mm_ThermalVias
- U1001, U1101, U1201, U1401, U1501, U1601, U1701, U1901, U2001, U2101, U2201, U2401, U2501, U2601, U2701, U2901, U3001, U301, U3101, U3201, U3401, U3501, U3601, U3701, U4301, U4401, U4501, U501, U601, U701, U901: footprint footprints:VCNT2025X01_VIS -> common:VCNT2025X01_VIS
- U1301, U1801, U2301, U2801, U3301, U3801, U401, U801: footprint footprints:WQFN16_RTE_TEX -> common:WQFN16_RTE_TEX
- U4: footprint footprints:DQA0010A -> common:DQA0010A
- U5: footprint footprints:QFN_24RGTR_TEX -> common:QFN_24RGTR_TEX
- U6: footprint footprints:SOT-563_DRL0006A -> common:SOT-563_DRL0006A
Changed lines of the file:
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@@
 		)
 	)
-	(footprint "footprints:VCNT2025X01_VIS"
+	(footprint "common:VCNT2025X01_VIS"
 		(layer "F.Cu")
 		(at 349.665799 2.4)
@@
 		(embedded_fonts no)
 	)
-	(footprint "footprints:MountingHole_2.7mm_M2.5_Keepout"
+	(footprint "common:MountingHole_2.7mm_M2.5_Keepout"
 		(layer "F.Cu")
 		(at 389.74 22.8)
@@
 		(embedded_fonts no)
 	)
-	(footprint "footprints:VCNT2025X01_VIS"
+	(footprint "common:VCNT2025X01_VIS"
 		(layer "F.Cu")
 		(at 162.999599 2.4)
@@
 		)
 	)
-	(footprint "footprints:VCNT2025X01_VIS"
+	(footprint "common:VCNT2025X01_VIS"
 		(layer "F.Cu")
 		(at 176.332899 2.4)
@@
 		)
 	)
-	(footprint "footprints:VCNT2025X01_VIS"
+	(footprint "common:VCNT2025X01_VIS"
 		(layer "F.Cu")
 		(at 229.6661 2.4)
@@
 		)
 	)
-	(footprint "footprints:VCNT2025X01_VIS"
+	(footprint "common:VCNT2025X01_VIS"
 		(layer "F.Cu")
 		(at 96.3331 2.4)
@@
 		)
 	)
-	(footprint "footprints:QFN_24RGTR_TEX"
+	(footprint "common:QFN_24RGTR_TEX"
 		(layer "F.Cu")
 		(at 158.525 18.925 -90)
@@
 		)
 	)
-	(footprint "footprints:MountingHole_2.7mm_M2.5_Keepout"
+	(footprint "common:MountingHole_2.7mm_M2.5_Keepout"
 		(layer "F.Cu")
 		(at 248.4 22.8)
@@
 		)
 	)
-	(footprint "footprints:VCNT2025X01_VIS"
+	(footprint "common:VCNT2025X01_VIS"
 		(layer "F.Cu")
 		(at 82.9998 2.4)
@@
 		)
 	)
-	(footprint "footprints:WQFN16_RTE_TEX"
+	(footprint "common:WQFN16_RTE_TEX"
 		(layer "F.Cu")
 		(at 363.25 13.025 180)
@@
 		(embedded_fonts no)
 	)
-	(footprint "footprints:WQFN16_RTE_TEX"
+	(footprint "common:WQFN16_RTE_TEX"
 		(layer "F.Cu")
 		(at 290.546 10.23 -90)
@@
 		)
 	)
-	(footprint "footprints:VCNT2025X01_VIS"
+	(footprint "common:VCNT2025X01_VIS"
 		(layer "F.Cu")
 		(at 29.6666 2.4)
@@
 		)
 	)
-	(footprint "footprints:VCNT2025X01_VIS"
+	(footprint "common:VCNT2025X01_VIS"
 		(layer "F.Cu")
 		(at 202.999499 2.4)
@@
 		)
 	)
-	(footprint "footprints:VCNT2025X01_VIS"
+	(footprint "common:VCNT2025X01_VIS"
 		(layer "F.Cu")
 		(at 149.6663 2.4)
@@
 		)
 	)
-	(footprint "footprints:VCNT2025X01_VIS"
+	(footprint "common:VCNT2025X01_VIS"
 		(layer "F.Cu")
 		(at 3 2.4)
@@
 		)
 	)
-	(footprint "footprints:SOT-563_DRL0006A"
+	(footprint "common:SOT-563_DRL0006A"
 		(layer "F.Cu")
 		(at 13.1 17.45)
@@
 		)
 	)
-	(footprint "footprints:mousebite_34mm"
+	(footprint "common:mousebite_34mm"
 		(locked yes)
 		(layer "F.Cu")
@@
 		(embedded_fonts no)
 	)
-	(footprint "footprints:C_0402_1005Metric_small_pads"
+	(footprint "common:C_0402_1005Metric_small_pads"
 		(layer "F.Cu")
 		(at 202.054348 19.366918 -135)
@@
 		)
 	)
-	(footprint "footprints:WQFN16_RTE_TEX"
+	(footprint "common:WQFN16_RTE_TEX"
 		(layer "F.Cu")
 		(at 178.56 10.23 -90)
@@
 		)
 	)
-	(footprint "footprints:MountingHole_2.7mm_M2.5_Keepout"
+	(footprint "common:MountingHole_2.7mm_M2.5_Keepout"
 		(layer "F.Cu")
 		(at 50 22.8)
@@
 		)
 	)
-	(footprint "footprints:VCNT2025X01_VIS"
+	(footprint "common:VCNT2025X01_VIS"
 		(layer "F.Cu")
 		(at 16.3333 2.4)
@@
 		(embedded_fonts no)
 	)
-	(footprint "footprints:WQFN16_RTE_TEX"
+	(footprint "common:WQFN16_RTE_TEX"
 		(layer "F.Cu")
 		(at 23.88 10.23 -90)
@@
 		)
 	)
-	(footprint "footprints:VCNT2025X01_VIS"
+	(footprint "common:VCNT2025X01_VIS"
 		(layer "F.Cu")
 		(at 296.3326 2.4)
@@
 		)
 	)
-	(footprint "footprints:MountingHole_2.7mm_M2.5_Keepout"
+	(footprint "common:MountingHole_2.7mm_M2.5_Keepout"
 		(layer "F.Cu")
 		(at 312.4 22.8)
@@
 		)
 	)
-	(footprint "footprints:MountingHole_2.7mm_M2.5_Keepout"
+	(footprint "common:MountingHole_2.7mm_M2.5_Keepout"
 		(layer "F.Cu")
 		(at 88.93 -4)
@@
 		)
 	)
-	(footprint "footprints:VCNT2025X01_VIS"
+	(footprint "common:VCNT2025X01_VIS"
 		(layer "F.Cu")
 		(at 122.9997 2.4)
@@
 		)
 	)
-	(footprint "footprints:VCNT2025X01_VIS"
+	(footprint "common:VCNT2025X01_VIS"
 		(layer "F.Cu")
 		(at 402.998999 2.4)
@@
 		)
 	)
-	(footprint "footprints:WQFN16_RTE_TEX"
+	(footprint "common:WQFN16_RTE_TEX"
 		(layer "F.Cu")
 		(at 230.4608 10.690001 -90)
@@
 		)
 	)
-	(footprint "footprints:WQFN16_RTE_TEX"
+	(footprint "common:WQFN16_RTE_TEX"
 		(layer "F.Cu")
 		(at 343.879199 10.23 -90)
@@
 		)
 	)
-	(footprint "footprints:VCNT2025X01_VIS"
+	(footprint "common:VCNT2025X01_VIS"
 		(layer "F.Cu")
 		(at 376.3324 2.4)
@@
 		)
 	)
-	(footprint "footprints:C_0402_1005Metric_small_pads"
+	(footprint "common:C_0402_1005Metric_small_pads"
 		(layer "F.Cu")
 		(at 202.747312 20.059883 -135)
@@
 		)
 	)
-	(footprint "footprints:VCNT2025X01_VIS"
+	(footprint "common:VCNT2025X01_VIS"
 		(layer "F.Cu")
 		(at 389.665699 2.4)
@@
 		)
 	)
-	(footprint "footprints:RP2350-QFN-60-1EP_7x7_P0.4mm_EP3.4x3.4mm_ThermalVias"
+	(footprint "common:RP2350-QFN-60-1EP_7x7_P0.4mm_EP3.4x3.4mm_ThermalVias"
 		(layer "F.Cu")
 		(at 200.237083 14.622232 -135)
@@
 		)
 	)
-	(footprint "footprints:VCNT2025X01_VIS"
+	(footprint "common:VCNT2025X01_VIS"
 		(layer "F.Cu")
 		(at 109.6664 2.4)
@@
 		)
 	)
-	(footprint "footprints:MountingHole_2.7mm_M2.5_Keepout"
+	(footprint "common:MountingHole_2.7mm_M2.5_Keepout"
 		(layer "F.Cu")
 		(at 155.21 -4)
@@
 		)
 	)
-	(footprint "footprints:MountingHole_2.7mm_M2.5_Keepout"
+	(footprint "common:MountingHole_2.7mm_M2.5_Keepout"
 		(layer "F.Cu")
 		(at 378.31 -4)
@@
 		)
 	)
-	(footprint "footprints:VCNT2025X01_VIS"
+	(footprint "common:VCNT2025X01_VIS"
 		(layer "F.Cu")
 		(at 309.6659 2.4)
@@
 		)
 	)
-	(footprint "footprints:MountingHole_2.7mm_M2.5_Keepout"
+	(footprint "common:MountingHole_2.7mm_M2.5_Keepout"
 		(layer "F.Cu")
 		(at 289.06 -4)
@@
 		(embedded_fonts no)
 	)
-	(footprint "footprints:MountingHole_2.7mm_M2.5_Keepout"
+	(footprint "common:MountingHole_2.7mm_M2.5_Keepout"
 		(layer "F.Cu")
 		(at 10.32 -4)
@@
 		)
 	)
-	(footprint "footprints:MountingHole_2.7mm_M2.5_Keepout"
+	(footprint "common:MountingHole_2.7mm_M2.5_Keepout"
 		(layer "F.Cu")
 		(at 389.47 -4)
@@
 		)
 	)
-	(footprint "footprints:MountingHole_2.7mm_M2.5_Keepout"
+	(footprint "common:MountingHole_2.7mm_M2.5_Keepout"
 		(layer "F.Cu")
 		(at 402.39 -4)
@@
 		(embedded_fonts no)
 	)
-	(footprint "footprints:VCNT2025X01_VIS"
+	(footprint "common:VCNT2025X01_VIS"
 		(layer "F.Cu")
 		(at 69.6665 2.4)
@@
 		)
 	)
-	(footprint "footprints:VCNT2025X01_VIS"
+	(footprint "common:VCNT2025X01_VIS"
 		(layer "F.Cu")
 		(at 42.9999 2.4)
@@
 		)
 	)
-	(footprint "footprints:VCNT2025X01_VIS"
+	(footprint "common:VCNT2025X01_VIS"
 		(layer "F.Cu")
 		(at 189.666199 2.4)
@@
 		)
 	)
-	(footprint "footprints:DQA0010A"
+	(footprint "common:DQA0010A"
 		(layer "F.Cu")
 		(at 5.025 19.435928 180)
@@
 		(embedded_fonts no)
 	)
-	(footprint "footprints:WQFN16_RTE_TEX"
+	(footprint "common:WQFN16_RTE_TEX"
 		(layer "F.Cu")
 		(at 130.5464 10.23 -90)
@@
 		)
 	)
-	(footprint "footprints:VCNT2025X01_VIS"
+	(footprint "common:VCNT2025X01_VIS"
 		(layer "F.Cu")
 		(at 216.3328 2.4)
@@
 		)
 	)
-	(footprint "footprints:SOD-323_L1.8-W1.3-LS2.5-RD"
+	(footprint "common:SOD-323_L1.8-W1.3-LS2.5-RD"
 		(layer "F.Cu")
 		(at 7.25 16 90)
@@
 		)
 	)
-	(footprint "footprints:VCNT2025X01_VIS"
+	(footprint "common:VCNT2025X01_VIS"
 		(layer "F.Cu")
 		(at 269.666 2.4)
@@
 		)
 	)
-	(footprint "footprints:VCNT2025X01_VIS"
+	(footprint "common:VCNT2025X01_VIS"
 		(layer "F.Cu")
 		(at 136.333 2.4)
@@
 		(embedded_fonts no)
 	)
-	(footprint "footprints:MountingHole_2.7mm_M2.5_Keepout"
+	(footprint "common:MountingHole_2.7mm_M2.5_Keepout"
 		(layer "F.Cu")
 		(at 106.55 22.8)
@@
 		)
 	)
-	(footprint "footprints:MountingHole_2.7mm_M2.5_Keepout"
+	(footprint "common:MountingHole_2.7mm_M2.5_Keepout"
 		(layer "F.Cu")
 		(at 364.97 22.8)
@@
 		(embedded_fonts no)
 	)
-	(footprint "footprints:VCNT2025X01_VIS"
+	(footprint "common:VCNT2025X01_VIS"
 		(layer "F.Cu")
 		(at 336.332499 2.4)
@@
 		)
 	)
-	(footprint "footprints:VCNT2025X01_VIS"
+	(footprint "common:VCNT2025X01_VIS"
 		(layer "F.Cu")
 		(at 282.9993 2.4)
@@
 		)
 	)
-	(footprint "footprints:VCNT2025X01_VIS"
+	(footprint "common:VCNT2025X01_VIS"
 		(layer "F.Cu")
 		(at 256.3327 2.4)
@@
 		(embedded_fonts no)
 	)
-	(footprint "footprints:L_pol_2016"
+	(footprint "common:L_pol_2016"
 		(layer "F.Cu")
 		(at 203.9 21.11 -135)
@@
 		)
 	)
-	(footprint "footprints:MountingHole_2.7mm_M2.5_Keepout"
+	(footprint "common:MountingHole_2.7mm_M2.5_Keepout"
 		(layer "F.Cu")
 		(at -1.45 8.825)
@@
 		)
 	)
-	(footprint "footprints:mousebite_34mm"
+	(footprint "common:mousebite_34mm"
 		(locked yes)
 		(layer "F.Cu")
@@
 		(embedded_fonts no)
 	)
-	(footprint "footprints:MountingHole_2.7mm_M2.5_Keepout"
+	(footprint "common:MountingHole_2.7mm_M2.5_Keepout"
 		(layer "F.Cu")
 		(at 378.79 22.8)
@@
 		)
 	)
-	(footprint "footprints:VCNT2025X01_VIS"
+	(footprint "common:VCNT2025X01_VIS"
 		(layer "F.Cu")
 		(at 362.999099 2.4)
@@
 		)
 	)
-	(footprint "footprints:VCNT2025X01_VIS"
+	(footprint "common:VCNT2025X01_VIS"
 		(layer "F.Cu")
 		(at 56.3332 2.4)
@@
 		)
 	)
-	(footprint "footprints:mousebite_34mm"
+	(footprint "common:mousebite_34mm"
 		(locked yes)
 		(layer "F.Cu")
@@
 		)
 	)
-	(footprint "footprints:MountingHole_2.7mm_M2.5_Keepout"
+	(footprint "common:MountingHole_2.7mm_M2.5_Keepout"
 		(layer "F.Cu")
 		(at 350.225 -4)
@@
 		)
 	)
-	(footprint "footprints:MountingHole_2.7mm_M2.5_Keepout"
+	(footprint "common:MountingHole_2.7mm_M2.5_Keepout"
 		(layer "F.Cu")
 		(at 402.35 22.8)
@@
 		)
 	)
-	(footprint "footprints:VCNT2025X01_VIS"
+	(footprint "common:VCNT2025X01_VIS"
 		(layer "F.Cu")
 		(at 322.999199 2.4)
@@
 		)
 	)
-	(footprint "footprints:MountingHole_2.7mm_M2.5_Keepout"
+	(footprint "common:MountingHole_2.7mm_M2.5_Keepout"
 		(layer "F.Cu")
 		(at 221.74 -4)
@@
 		)
 	)
-	(footprint "footprints:VCNT2025X01_VIS"
+	(footprint "common:VCNT2025X01_VIS"
 		(layer "F.Cu")
 		(at 242.9994 2.4)
@@
 		)
 	)
-	(footprint "footprints:WQFN16_RTE_TEX"
+	(footprint "common:WQFN16_RTE_TEX"
 		(layer "F.Cu")
 		(at 77.2132 10.23 -90)
