File: hardware/kicad/002_sensor_board/002_Sensor_PI_RS485 board.kicad_pcb (KiCad board)
At the start: 2 copper layers, 413.7 x 35 mm, 300 parts, among them J1 JST_SH, J2 JST_SH, J3 USB_C_Receptacle_USB2.0, Q1001 AO3400A, Q1101 AO3400A, Q1201 AO3400A, Q1401 AO3400A, Q1501 AO3400A, Q1601 AO3400A, Q1701 AO3400A, Q1901 AO3400A, Q2001 AO3400A, Q2101 AO3400A, Q2201 AO3400A, Q2401 AO3400A, Q2501 AO3400A, Q2601 AO3400A, Q2701 AO3400A, Q2901 AO3400A, Q3001 AO3400A, Q301 AO3400A, Q3101 AO3400A, Q3201 AO3400A, Q3401 AO3400A, Q3501 AO3400A, Q3601 AO3400A, Q3701 AO3400A, Q4301 AO3400A, Q4401 AO3400A, Q4501 AO3400A, Q501 AO3400A, Q601 AO3400A, Q701 AO3400A, Q901 AO3400A, U1 RP2354_60QFN, U1001 VCNT2025X01, U1101 VCNT2025X01, U1201 VCNT2025X01, U1301 TLA2518IRTER, U1401 VCNT2025X01, U1501 VCNT2025X01, U1601 VCNT2025X01, U1701 VCNT2025X01, U1801 TLA2518IRTER, U1901 VCNT2025X01, U2001 VCNT2025X01, U2101 VCNT2025X01, U2201 VCNT2025X01, U2301 TLA2518IRTER, U2401 VCNT2025X01, U2501 VCNT2025X01, U2601 VCNT2025X01, U2701 VCNT2025X01, U2801 TLA2518IRTER, U2901 VCNT2025X01, U3001 VCNT2025X01, U301 VCNT2025X01, U3101 VCNT2025X01, U3201 VCNT2025X01, U3301 TLA2518IRTER, U3401 VCNT2025X01, U3501 VCNT2025X01, U3601 VCNT2025X01, U3701 VCNT2025X01, U3801 TLA2518IRTER, U4 TPD4E05U06DQAR, U401 TLA2518IRTER, U4301 VCNT2025X01, U4401 VCNT2025X01, U4501 VCNT2025X01, U5 THVD1424RGTR, U501 VCNT2025X01, U6 TPS62A0569ADRLR, U601 VCNT2025X01, U701 VCNT2025X01, U801 TLA2518IRTER, U901 VCNT2025X01, Y1 ABM8-272-T3

Commit message: Rename shared footprint library common -> photon_common
'common' is too generic for a library nickname - it can collide with a
global library or another project's table, and it doesn't identify whose
footprints these are.

155 lib_ids rewritten across the three boards plus all three
fp-lib-tables. All 459 footprint references still resolve.

Co-Authored-By: Claude Opus 5 <noreply@anthropic.com>
Parts:
- C2, C3: footprint common:C_0402_1005Metric_small_pads -> photon_common:C_0402_1005Metric_small_pads
- CR1: footprint common:SOD-323_L1.8-W1.3-LS2.5-RD -> photon_common:SOD-323_L1.8-W1.3-LS2.5-RD
- H1, H10, H11, H12, H13, H14, H15, H16, H17, H18, H2, H3, H4, H5, H6, H7, H8, H9: footprint common:MountingHole_2.7mm_M2.5_Keepout -> photon_common:MountingHole_2.7mm_M2.5_Keepout
- H3801, H3802, H3803: footprint common:mousebite_34mm -> photon_common:mousebite_34mm
- L1: footprint common:L_pol_2016 -> photon_common:L_pol_2016
- U1: footprint common:RP2350-QFN-60-1EP_7x7_P0.4mm_EP3.4x3.4mm_ThermalVias -> photon_common:RP2350-QFN-60-1EP_7x7_P0.4mm_EP3.4x3.4mm_ThermalVias
- U1001, U1101, U1201, U1401, U1501, U1601, U1701, U1901, U2001, U2101, U2201, U2401, U2501, U2601, U2701, U2901, U3001, U301, U3101, U3201, U3401, U3501, U3601, U3701, U4301, U4401, U4501, U501, U601, U701, U901: footprint common:VCNT2025X01_VIS -> photon_common:VCNT2025X01_VIS
- U1301, U1801, U2301, U2801, U3301, U3801, U401, U801: footprint common:WQFN16_RTE_TEX -> photon_common:WQFN16_RTE_TEX
- U4: footprint common:DQA0010A -> photon_common:DQA0010A
- U5: footprint common:QFN_24RGTR_TEX -> photon_common:QFN_24RGTR_TEX
- U6: footprint common:SOT-563_DRL0006A -> photon_common:SOT-563_DRL0006A
