File: hardware/kicad/002_sensor_board/Indiv_sensor.kicad_sch (KiCad schematic)
At the start: 5 parts, among them Q301 AO3400A, U301 VCNT2025X01

Commit message: Consolidate footprints into a single shared library
All three boards carried their own copies of the same footprints - 79
files across 11 project libraries for 37 distinct footprints. Several
existed three times over (RP2350-QFN-60 ThermalVias, edge_holes,
TO-236_VIS-L, SON_NT2020_VIS, L_pol_2016, USB_Micro-B). Three copies
drift, and this project has already been bitten twice by a library and
a board disagreeing.

- New hardware/kicad/common.pretty holds all 37, verified byte-identical
  where they were duplicated: zero name collisions with differing
  content, so nothing had to be reconciled.
- Each board's fp-lib-table is now a single "common" entry. Previously
  001 alone had eight, and the nickname "footprints" meant a different
  library on each of the three boards - so lib_ids were rewritten per
  board, not globally.
- 459 footprint references across the three boards now resolve. That
  includes SparkFun-Qwiic:qwiic_8mm on 001, which was referenced but
  had never been in any fp-lib-table - broken before this change.

Also shrinks docs/images/reflective_sensor.png from 2816x1536 / 4.43 MB
to 1600x873 / 1.72 MB.

Co-Authored-By: Claude Opus 5 <noreply@anthropic.com>
Parts:
- U301: footprint footprints:VCNT2025X01_VIS -> common:VCNT2025X01_VIS
Changed lines of the file:
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@@
 			)
 		)
-		(property "Footprint" "footprints:VCNT2025X01_VIS"
+		(property "Footprint" "common:VCNT2025X01_VIS"
 			(at 138.43 102.87 0)
 			(hide yes)

Commit message: Rename shared footprint library common -> photon_common
'common' is too generic for a library nickname - it can collide with a
global library or another project's table, and it doesn't identify whose
footprints these are.

155 lib_ids rewritten across the three boards plus all three
fp-lib-tables. All 459 footprint references still resolve.

Co-Authored-By: Claude Opus 5 <noreply@anthropic.com>
Parts:
- U301: footprint common:VCNT2025X01_VIS -> photon_common:VCNT2025X01_VIS
Changed lines of the file:
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@@
 			)
 		)
-		(property "Footprint" "common:VCNT2025X01_VIS"
+		(property "Footprint" "photon_common:VCNT2025X01_VIS"
 			(at 138.43 102.87 0)
 			(hide yes)
