File: hardware/kicad/002_sensor_board/4_Sensor_Bank.kicad_sch (KiCad schematic)
At the start: 8 parts, among them U401 TLA2518IRTER

Commit message: Consolidate footprints into a single shared library
All three boards carried their own copies of the same footprints - 79
files across 11 project libraries for 37 distinct footprints. Several
existed three times over (RP2350-QFN-60 ThermalVias, edge_holes,
TO-236_VIS-L, SON_NT2020_VIS, L_pol_2016, USB_Micro-B). Three copies
drift, and this project has already been bitten twice by a library and
a board disagreeing.

- New hardware/kicad/common.pretty holds all 37, verified byte-identical
  where they were duplicated: zero name collisions with differing
  content, so nothing had to be reconciled.
- Each board's fp-lib-table is now a single "common" entry. Previously
  001 alone had eight, and the nickname "footprints" meant a different
  library on each of the three boards - so lib_ids were rewritten per
  board, not globally.
- 459 footprint references across the three boards now resolve. That
  includes SparkFun-Qwiic:qwiic_8mm on 001, which was referenced but
  had never been in any fp-lib-table - broken before this change.

Also shrinks docs/images/reflective_sensor.png from 2816x1536 / 4.43 MB
to 1600x873 / 1.72 MB.

Co-Authored-By: Claude Opus 5 <noreply@anthropic.com>
Parts:
- U401: footprint footprints:WQFN16_RTE_TEX -> common:WQFN16_RTE_TEX
Changed lines of the file:
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@@
 			)
 		)
-		(property "Footprint" "footprints:WQFN16_RTE_TEX"
+		(property "Footprint" "common:WQFN16_RTE_TEX"
 			(at 93.98 120.65 0)
 			(hide yes)

Commit message: Rename shared footprint library common -> photon_common
'common' is too generic for a library nickname - it can collide with a
global library or another project's table, and it doesn't identify whose
footprints these are.

155 lib_ids rewritten across the three boards plus all three
fp-lib-tables. All 459 footprint references still resolve.

Co-Authored-By: Claude Opus 5 <noreply@anthropic.com>
Parts:
- U401: footprint common:WQFN16_RTE_TEX -> photon_common:WQFN16_RTE_TEX
Changed lines of the file:
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@@
 			)
 		)
-		(property "Footprint" "common:WQFN16_RTE_TEX"
+		(property "Footprint" "photon_common:WQFN16_RTE_TEX"
 			(at 93.98 120.65 0)
 			(hide yes)

Commit message: Consolidate symbol libraries, normalise BOM data, Rev B for all three boards
Libraries
- Move PHOTON and PHOTON_Modified to hardware/kicad/, shared by all three
  projects, replacing six divergent per-project copies. 002's versions taken
  as canonical (correct pin electrical types); 001-only parts recovered from
  the schematic cache. All 459 footprint and 464 symbol refs resolve.
- Repoint every sym-lib-table at the shared files. Nicknames unchanged, so
  002 and 001d needed no lib_id edits; only 001's stale date-named ones.
- Fix stale footprint nicknames inside the symbol libraries (footprints:,
  RP2350_60QFN_minimal:, APS6404L-3SQR-ZR:) that would have made newly
  placed parts land with unresolvable footprints.
- Reset baked-in reference designators and MPNs on six library footprints
  back to REF** and the footprint name. SOT-563_DRL0006A carried "U6",
  which would have overwritten 001d's U5 on any field-resetting update.

Footprints
- Add SON-8_3x2mm_P0.5mm: KiCad stock SON-8 with the exposed pad and its
  four paste apertures removed. The APS6404L USON-8L (JEDEC MO-229) has no
  thermal pad and 0-0.05mm standoff, so both the copper and the paste under
  the body were wrong. Replaces the easyeda2kicad footprint on U101, whose
  0.102mm mask margin also bridged all six 0.5mm-pitch mask openings.
- Mounting holes on 001 and 001d move to the photon_common keepout
  footprint, matching 002, so a screw head cannot bridge the F.Cu power
  pour to the B.Cu ground pour.
- Remove the unused TDK T3902 microphone footprint.

BOM
- Normalise values fleet-wide: Greek mu -> ascii u, strip spaces before
  units, complete truncated inductor values. Each was splitting one part
  into two BOM lines, since the fab toolkit groups on footprint+value.
- Unify JST-SH connector values so each board emits one line, not three.
  Per-connector labels moved to Description, which is not a BOM column.
- Assign part numbers to the four largest passive lines: 100nF C1525,
  1uF C52923, 1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
Parts:
- C401, C402, C403: JLCPCB Part # (none) -> C52923
- C404, C405, C406, C407: JLCPCB Part # (none) -> C1523
Changed lines of the file:
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@@
+			)
+		)
+		(property "JLCPCB Part #" "C52923"
+			(at 168.91 149.86 0)
+			(show_name no)
+			(do_not_autoplace no)
+			(hide yes)
+			(effects
+				(font
+					(size 1.27 1.27)
+				)
 			)
 		)
@@
 			(show_name no)
 			(do_not_autoplace no)
+			(effects
+				(font
+					(size 1.27 1.27)
+				)
+			)
+		)
+		(property "JLCPCB Part #" "C52923"
+			(at 92.71 142.24 0)
+			(show_name no)
+			(do_not_autoplace no)
+			(hide yes)
 			(effects
 				(font
@@
 			)
 		)
+		(property "JLCPCB Part #" "C1523"
+			(at 201.93 128.27 0)
+			(show_name no)
+			(do_not_autoplace no)
+			(hide yes)
+			(effects
+				(font
+					(size 1.27 1.27)
+				)
+			)
+		)
 		(property "Description" "Unpolarized capacitor"
 			(at 201.93 128.27 0)
@@
 			)
 		)
+		(property "JLCPCB Part #" "C1523"
+			(at 229.87 128.27 0)
+			(show_name no)
+			(do_not_autoplace no)
+			(hide yes)
+			(effects
+				(font
+					(size 1.27 1.27)
+				)
+			)
+		)
 		(property "Description" "Unpolarized capacitor"
 			(at 229.87 128.27 0)
@@
 			)
 		)
+		(property "JLCPCB Part #" "C1523"
+			(at 215.9 128.27 0)
+			(show_name no)
+			(do_not_autoplace no)
+			(hide yes)
+			(effects
+				(font
+					(size 1.27 1.27)
+				)
+			)
+		)
 		(property "Description" "Unpolarized capacitor"
 			(at 215.9 128.27 0)
@@
 			)
 		)
+		(property "JLCPCB Part #" "C1523"
+			(at 242.57 128.27 0)
+			(show_name no)
+			(do_not_autoplace no)
+			(hide yes)
+			(effects
+				(font
+					(size 1.27 1.27)
+				)
+			)
+		)
 		(property "Description" "Unpolarized capacitor"
 			(at 242.57 128.27 0)
@@
 			(effects
 				(font
+					(size 1.27 1.27)
+				)
+			)
+		)
+		(property "JLCPCB Part #" "C52923"
+			(at 81.28 142.24 0)
+			(show_name no)
+			(do_not_autoplace no)
+			(hide yes)
+			(effects
+				(font
