File: hardware/kicad/002_sensor_board/002_Sensor_PI_RS485 board.kicad_sch (KiCad schematic)
At the start: 79 parts, among them J1 JST_SH, J2 JST_SH, J3 USB_C_Receptacle_USB2.0, U1 RP2354_60QFN, U4 TPD4E05U06DQAR, U5 THVD1424RGTR, U6 TPS62A0569ADRLR, Y1 ABM8-272-T3

Commit message: Consolidate symbol libraries, normalise BOM data, Rev B for all three boards
Libraries
- Move PHOTON and PHOTON_Modified to hardware/kicad/, shared by all three
  projects, replacing six divergent per-project copies. 002's versions taken
  as canonical (correct pin electrical types); 001-only parts recovered from
  the schematic cache. All 459 footprint and 464 symbol refs resolve.
- Repoint every sym-lib-table at the shared files. Nicknames unchanged, so
  002 and 001d needed no lib_id edits; only 001's stale date-named ones.
- Fix stale footprint nicknames inside the symbol libraries (footprints:,
  RP2350_60QFN_minimal:, APS6404L-3SQR-ZR:) that would have made newly
  placed parts land with unresolvable footprints.
- Reset baked-in reference designators and MPNs on six library footprints
  back to REF** and the footprint name. SOT-563_DRL0006A carried "U6",
  which would have overwritten 001d's U5 on any field-resetting update.

Footprints
- Add SON-8_3x2mm_P0.5mm: KiCad stock SON-8 with the exposed pad and its
  four paste apertures removed. The APS6404L USON-8L (JEDEC MO-229) has no
  thermal pad and 0-0.05mm standoff, so both the copper and the paste under
  the body were wrong. Replaces the easyeda2kicad footprint on U101, whose
  0.102mm mask margin also bridged all six 0.5mm-pitch mask openings.
- Mounting holes on 001 and 001d move to the photon_common keepout
  footprint, matching 002, so a screw head cannot bridge the F.Cu power
  pour to the B.Cu ground pour.
- Remove the unused TDK T3902 microphone footprint.

BOM
- Normalise values fleet-wide: Greek mu -> ascii u, strip spaces before
  units, complete truncated inductor values. Each was splitting one part
  into two BOM lines, since the fab toolkit groups on footprint+value.
- Unify JST-SH connector values so each board emits one line, not three.
  Per-connector labels moved to Description, which is not a BOM column.
- Assign part numbers to the four largest passive lines: 100nF C1525,
  1uF C52923, 1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
Parts:
- C10: JLCPCB Part # (none) -> C52923
- C13, C14, C15, C16, C19, C20, C21, C22, C23, C24, C25, C26, C27, C5, C8, C9: JLCPCB Part # (none) -> C1525
- C17, C18: JLCPCB Part # (none) -> C1548
Changed lines of the file:
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@@
 			)
 		)
+		(property "JLCPCB Part #" "C1525"
+			(at 72.39 236.22 0)
+			(show_name no)
+			(do_not_autoplace no)
+			(hide yes)
+			(effects
+				(font
+					(size 1.27 1.27)
+				)
+			)
+		)
 		(property "Description" ""
 			(at 72.39 236.22 0)
@@
 			)
 		)
+		(property "JLCPCB Part #" "C1525"
+			(at 106.68 236.22 0)
+			(show_name no)
+			(do_not_autoplace no)
+			(hide yes)
+			(effects
+				(font
+					(size 1.27 1.27)
+				)
+			)
+		)
 		(property "Description" ""
 			(at 106.68 236.22 0)
@@
 			)
 		)
+		(property "JLCPCB Part #" "C1525"
+			(at 60.96 236.22 0)
+			(show_name no)
+			(do_not_autoplace no)
+			(hide yes)
+			(effects
+				(font
+					(size 1.27 1.27)
+				)
+			)
+		)
 		(property "Description" ""
 			(at 60.96 236.22 0)
@@
 			)
 		)
+		(property "JLCPCB Part #" "C1525"
+			(at 320.04 29.21 0)
+			(show_name no)
+			(do_not_autoplace no)
+			(hide yes)
+			(effects
+				(font
+					(size 1.27 1.27)
+				)
+			)
+		)
 		(property "Description" ""
 			(at 320.04 29.21 0)
@@
 			)
 		)
+		(property "JLCPCB Part #" "C1525"
+			(at 83.82 236.22 0)
+			(show_name no)
+			(do_not_autoplace no)
+			(hide yes)
+			(effects
+				(font
+					(size 1.27 1.27)
+				)
+			)
+		)
 		(property "Description" ""
 			(at 83.82 236.22 0)
@@
 			)
 		)
+		(property "JLCPCB Part #" "C1525"
+			(at 365.76 29.21 0)
+			(show_name no)
+			(do_not_autoplace no)
+			(hide yes)
+			(effects
+				(font
+					(size 1.27 1.27)
+				)
+			)
+		)
 		(property "Description" ""
 			(at 365.76 29.21 0)
@@
 			)
 		)
+		(property "JLCPCB Part #" "C1548"
+			(at 332.74 187.96 0)
+			(show_name no)
+			(do_not_autoplace no)
+			(hide yes)
+			(effects
+				(font
+					(size 1.27 1.27)
+				)
+			)
+		)
 		(property "Description" ""
 			(at 332.74 187.96 0)
@@
 			)
 		)
+		(property "JLCPCB Part #" "C1525"
+			(at 234.95 245.11 0)
+			(show_name no)
+			(do_not_autoplace no)
+			(hide yes)
+			(effects
+				(font
+					(size 1.27 1.27)
+				)
+			)
+		)
 		(property "Description" ""
 			(at 234.95 245.11 0)
@@
 			)
 		)
+		(property "JLCPCB Part #" "C1525"
+			(at 354.33 29.21 0)
+			(show_name no)
+			(do_not_autoplace no)
+			(hide yes)
+			(effects
+				(font
+					(size 1.27 1.27)
+				)
+			)
+		)
 		(property "Description" ""
 			(at 354.33 29.21 0)
@@
 			)
 		)
+		(property "JLCPCB Part #" "C1525"
+			(at 308.61 29.21 0)
+			(show_name no)
+			(do_not_autoplace no)
+			(hide yes)
+			(effects
+				(font
+					(size 1.27 1.27)
+				)
+			)
+		)
 		(property "Description" ""
 			(at 308.61 29.21 0)
@@
 			)
 		)
+		(property "JLCPCB Part #" "C1525"
+			(at 377.19 29.21 0)
+			(show_name no)
+			(do_not_autoplace no)
+			(hide yes)
+			(effects
+				(font
+					(size 1.27 1.27)
+				)
+			)
+		)
 		(property "Description" ""
 			(at 377.19 29.21 0)
@@
 			)
 		)
+		(property "JLCPCB Part #" "C1525"
+			(at 228.6 29.21 0)
+			(show_name no)
+			(do_not_autoplace no)
+			(hide yes)
+			(effects
+				(font
+					(size 1.27 1.27)
+				)
+			)
+		)
 		(property "Description" ""
 			(at 228.6 29.21 0)
@@
 			)
 		)
+		(property "JLCPCB Part #" "C1525"
+			(at 49.53 236.22 0)
+			(show_name no)
+			(do_not_autoplace no)
+			(hide yes)
+			(effects
+				(font
+					(size 1.27 1.27)
+				)
+			)
+		)
 		(property "Description" ""
 			(at 49.53 236.22 0)
@@
 			)
 		)
+		(property "JLCPCB Part #" "C1525"
+			(at 342.9 29.21 0)
+			(show_name no)
+			(do_not_autoplace no)
+			(hide yes)
+			(effects
+				(font
+					(size 1.27 1.27)
+				)
+			)
+		)
 		(property "Description" ""
 			(at 342.9 29.21 0)
@@
 			)
 		)
+		(property "JLCPCB Part #" "C52923"
+			(at 247.65 245.11 0)
+			(show_name no)
+			(do_not_autoplace no)
+			(hide yes)
+			(effects
+				(font
+					(size 1.27 1.27)
+				)
+			)
+		)
 		(property "Description" ""
 			(at 247.65 245.11 0)
@@
 			)
 		)
+		(property "JLCPCB Part #" "C1525"
+			(at 95.25 236.22 0)
+			(show_name no)
+			(do_not_autoplace no)
+			(hide yes)
+			(effects
+				(font
+					(size 1.27 1.27)
+				)
+			)
+		)
 		(property "Description" ""
 			(at 95.25 236.22 0)
@@
 			)
 		)
+		(property "JLCPCB Part #" "C1525"
+			(at 251.46 29.21 0)
+			(show_name no)
+			(do_not_autoplace no)
+			(hide yes)
+			(effects
+				(font
+					(size 1.27 1.27)
+				)
+			)
+		)
 		(property "Description" ""
 			(at 251.46 29.21 0)
@@
 			)
 		)
+		(property "JLCPCB Part #" "C1525"
+			(at 331.47 29.21 0)
+			(show_name no)
+			(do_not_autoplace no)
+			(hide yes)
+			(effects
+				(font
+					(size 1.27 1.27)
+				)
+			)
+		)
 		(property "Description" ""
 			(at 331.47 29.21 0)
@@
 			(effects
 				(font
+					(size 1.27 1.27)
+				)
+			)
+		)
+		(property "JLCPCB Part #" "C1548"
+			(at 332.74 177.8 0)
+			(show_name no)
+			(do_not_autoplace no)
+			(hide yes)
+			(effects
+				(font

Commit message: Pin the 4.7uF 0402 to C23733 across all three boards
JLCPCB selected Samsung CL05A475MP5NRNC (4.7uF 10V X5R +/-20% 0402) for the
blank 4.7uF line when 001d and 002 were ordered. Recording it so the choice is
deterministic on the next order rather than made again at upload time, possibly
differently.

Matched on value AND footprint: the twelve 0402 parts (C2/C3/C6/C7 on each
board, across both the standard and small-pads variants) take C23733, while
C1 — the 4.7uF 0805 at the buck input — keeps C1779.

10 V is the right side of the choice for a 3.3 V rail; a 6.3 V part would
derate much harder under bias. These four are bypass and the low-bias +1V1
core rail, not the buck's control loop, which hangs off C4 (22uF 0805).

Co-Authored-By: Claude Opus 5 <noreply@anthropic.com>
Parts:
- C2, C3, C6, C7: JLCPCB Part # (none) -> C23733
Changed lines of the file:
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@@
 			)
 		)
+		(property "JLCPCB Part #" "C23733"
+			(at 0 0 0)
+			(show_name no)
+			(do_not_autoplace no)
+			(hide yes)
+			(effects
+				(font
+					(size 1.27 1.27)
+				)
+			)
+		)
 		(property "Description" ""
 			(at 240.03 29.21 0)
@@
 			)
 		)
+		(property "JLCPCB Part #" "C23733"
+			(at 0 0 0)
+			(show_name no)
+			(do_not_autoplace no)
+			(hide yes)
+			(effects
+				(font
+					(size 1.27 1.27)
+				)
+			)
+		)
 		(property "Description" ""
 			(at 193.04 67.31 0)
@@
 			)
 		)
+		(property "JLCPCB Part #" "C23733"
+			(at 0 0 0)
+			(show_name no)
+			(do_not_autoplace no)
+			(hide yes)
+			(effects
+				(font
+					(size 1.27 1.27)
+				)
+			)
+		)
 		(property "Description" ""
 			(at 238.76 54.61 0)
@@
 			(effects
 				(font
+					(size 1.27 1.27)
+				)
+			)
+		)
+		(property "JLCPCB Part #" "C23733"
+			(at 0 0 0)
+			(show_name no)
+			(do_not_autoplace no)
+			(hide yes)
+			(effects
+				(font
