File: hardware/kicad/001d_main_controller_board_low_profile/PHOTON_main_controller_1d.kicad_sch (KiCad schematic)
At the start: 63 parts, among them J101 JST_SH, J102 JST_SH, J103 JST_SH, J3 USB_C_Receptacle_USB2.0, J4 Micro_SD_Card, U1 RP2354_60QFN, U102 THVD1424RGTR, U4 TPD4E05U06DQAR, U5 TPS62A0569ADRLR, Y1 ABM8-272-T3

Commit message: Pin the 4.7uF 0402 to C23733 across all three boards
JLCPCB selected Samsung CL05A475MP5NRNC (4.7uF 10V X5R +/-20% 0402) for the
blank 4.7uF line when 001d and 002 were ordered. Recording it so the choice is
deterministic on the next order rather than made again at upload time, possibly
differently.

Matched on value AND footprint: the twelve 0402 parts (C2/C3/C6/C7 on each
board, across both the standard and small-pads variants) take C23733, while
C1 — the 4.7uF 0805 at the buck input — keeps C1779.

10 V is the right side of the choice for a 3.3 V rail; a 6.3 V part would
derate much harder under bias. These four are bypass and the low-bias +1V1
core rail, not the buck's control loop, which hangs off C4 (22uF 0805).

Co-Authored-By: Claude Opus 5 <noreply@anthropic.com>
Parts:
- C2, C3, C6, C7: JLCPCB Part # (none) -> C23733
Changed lines of the file:
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@@
 			)
 		)
+		(property "JLCPCB Part #" "C23733"
+			(at 0 0 0)
+			(show_name no)
+			(do_not_autoplace no)
+			(hide yes)
+			(effects
+				(font
+					(size 1.27 1.27)
+				)
+			)
+		)
 		(property "Description" ""
 			(at 237.49 29.21 0)
@@
 			)
 		)
+		(property "JLCPCB Part #" "C23733"
+			(at 0 0 0)
+			(show_name no)
+			(do_not_autoplace no)
+			(hide yes)
+			(effects
+				(font
+					(size 1.27 1.27)
+				)
+			)
+		)
 		(property "Description" ""
 			(at 190.5 67.31 0)
@@
 			)
 		)
+		(property "JLCPCB Part #" "C23733"
+			(at 0 0 0)
+			(show_name no)
+			(do_not_autoplace no)
+			(hide yes)
+			(effects
+				(font
+					(size 1.27 1.27)
+				)
+			)
+		)
 		(property "Description" ""
 			(at 236.22 54.61 0)
@@
 			(effects
 				(font
+					(size 1.27 1.27)
+				)
+			)
+		)
+		(property "JLCPCB Part #" "C23733"
+			(at 0 0 0)
+			(show_name no)
+			(do_not_autoplace no)
+			(hide yes)
+			(effects
+				(font
